File: ACC-MB/Rev0/ACC-MB-R0.sch (EAGLE design)
At the start: 0 parts

Commit message: mobo update
Parts:
- added 1A_500V_FUSE_ENERGYMETER, 1A_500V_FUSE_IMD_VSENSE, HV+_FUSE_DRY: _CUSTOM_PARTS_LF_885, _CUSTOM:_CUSTOM_PARTS_LF_885
- added AMS, DISCH, IMD, MONITOR, SPR1, SPR2: 3568FUSEHOLDER, fuse:3568FUSEHOLDER
- added C1: 39n, resistor:C-USC0805
- added C2: 10n, resistor:C-USC0805
- added C3: 100n, resistor:C-USC0805
- added C4: 4.7u, resistor:C-USC0805
- added C5: 0.1u, resistor:C-USC0805
- added CFILTER_1, CFILTER_2: 3uF, _CUSTOM:B58035U5305M062
- added COUT_EXT: (no value), resistor:CPOL-USE7.5-16
- added D1, D4: 1N4004, diode:1N4004
- added D2: 1N4758A - 56Vz, diode:ZENER-DIODEZD-12.5
- added DCM290P138T600A40: 600W 400 to 12V, 111_Custom:VICOR_CHIP_WITH_HEATSINK
- added H1, H2, H3, H4, H5, H6: MOUNT-HOLE3.3, holes:MOUNT-HOLE3.3
- added IC1: 555, SparkFun-IC-Special-Function:555P
- added IC2: NUD3124DMT1G, _CUSTOM:SAMACSYS_PARTS_NUD3124DMT1G
- added INPUT_FUSE: 2.5A, _CUSTOM:_CUSTOM_PARTS_LF_885
- added L_IN: 39uH, _CUSTOM:SRP1770TA-390M
- added OK3: LTV816, optocoupler:LTV816
- added R1, R3, R5, R7: 100, resistor:R-US_R0805
- added R10: 4.7M, resistor:R-US_R0805
- added R11, R2, R4, R6, R8: 1M, resistor:R-US_R0805
- added R12: (no value), rcl:R-EU_R0805
- added R13, R14, R15: (no value), rcl:R-US_R0805
- added R16: 200, rcl:R-US_R2010
- added R17, R19: 10k, resistor:R-US_R0805
- added R9: 2.2k, resistor:R-US_R0805
- added R_IN: 2.5, resistor-power:RMG100-V
- added U$1: PHOENIX_1935789, _CUSTOM:PHOENIX_1935789
- added U$10, U$11, U$12, U$13, U$14: BUZ11, transistor-fet:BUZ11
- added U$15: MIC4417, HVIB_v2:MIC4417
- added U$16, U$17: DCDC_PARTS_282838-2_TE, _CUSTOM:DCDC_PARTS_282838-2_TE
- added U$18: UCC27511AQDBVRQ1, _CUSTOM:UCC27511AQDBVRQ1
- added U$19: _CUSTOM_IXCY10M90SD2PAK, HVIB_v2:_CUSTOM_IXCY10M90SD2PAK
- added U$2, U$3: HSA25, 111_Custom:HSA25
- added U$20, U$21, U$22: _CUSTOM_111_CUSTOM_SQJ407EP-T1_GE3, PDM_2019_RevB:_CUSTOM_111_CUSTOM_SQJ407EP-T1_GE3
- added U$23, U$25: 1777642_PHOENIX, CUSTOM_PARTS:1777642_PHOENIX
- added U$24: TO247RESISTORHEATINK, 111:TO247RESISTORHEATINK
- added U$26: DTM1312PA12BR008, CUSTOM_PARTS:DTM1312PA12BR008
- added U$27, U$28, U$29, U$30: SR4M4012_TE, CUSTOM_PARTS:SR4M4012_TE
- added U$4: G7L, precharge:G7L
- added U$5, U$6: 1935200_PHOENIX, DCDC_Parts:1935200_PHOENIX
- added U$7: PHOENIX_1725724, 111_Custom:PHOENIX_1725724
- added U$8: RK7002BMT116, 111_Custom:RK7002BMT116
- added U$9: 1777600_PHOENIX, DCDC_Parts:1777600_PHOENIX
- added X1: PRECH_IN, con-phoenix-350:1751248
Connections:
- new net +12V: AMS.1A, AMS.1B, C3.1, C4.1, C5.1, DISCH.1A, DISCH.1B, IC1./RES, IC1.VCC+, IMD.1A, IMD.1B, MONITOR.1A, MONITOR.1B, OK3.COL, R11.2, R9.2, SPR1.1A, SPR1.1B, SPR2.1A, SPR2.1B, U$1.3, U$15.VS, U$18.IN+, U$18.VDD, U$20.D, U$21.D, U$22.D, U$23.P$10, U$25.P$1, U$25.P$3, U$26.P$1, U$26.P$21, U$26.P$3, U$27.NOA3, U$4.1, U$7.P$1, U$7.P$3, U$7.P$6, U$9.P$5, U$9.P$6, U$9.P$7, U$9.P$8
- new net ACC_LGHT: U$10.D, U$7.P$7
- new net AIR_ON: D1.C, D4.C, R19.2, R5.1, R6.2, U$10.G, U$15.CTL
- new net AMS+: AMS.2A, AMS.2B, U$5.P$3
- new net CH1IN: U$25.P$2, U$25.P$5, U$26.P$2, U$26.P$5, U$27.NOA2
- new net CH2IN: U$25.P$4, U$25.P$7, U$26.P$4, U$26.P$7, U$28.NOB2
- new net CTRL: IC2.G1, IC2.G2, U$1.2
- new net DCDC_OUT: COUT_EXT.+, DCM290P138T600A40.OUT+_1, DCM290P138T600A40.OUT+_2, R15.1, U$20.S, U$21.S, U$22.S
- new net DISCHPWR: DISCH.2A, DISCH.2B, U$6.P$1
- new net GND: C1.2, C2.2, C3.2, C4.2, C5.2, COUT_EXT.-, DCM290P138T600A40.OUT-_1, DCM290P138T600A40.OUT-_2, IC1.GND, R12.1, R13.1, R17.1, R19.1, R2.1, R4.1, R6.1, R8.1, U$10.S, U$11.S, U$12.S, U$14.S, U$15.GND, U$18.GND, U$23.P$9, U$26.P$22, U$27.COIL+, U$28.COIL-, U$29.COIL+, U$30.COIL+, U$5.P$2, U$5.P$4, U$5.P$6, U$6.P$2, U$6.P$4, U$6.P$6, U$7.P$2, U$8.S, U$9.P$1, U$9.P$2, U$9.P$3, U$9.P$4
- new net GNDA: IC2.S1, IC2.S2, U$1.1
- new net HV+_DRY_FUSED: D2.C, HV+_FUSE_DRY.P$1
- new net HV+_WET: U$24.P$2
- new net HV-_DRY: OK3.C
- new net IMD+: IMD.2A, IMD.2B, U$5.P$1
- new net MON+: MONITOR.2A, MONITOR.2B, U$5.P$5
- new net N$1: R1.1, R2.2
- new net N$10: D2.A, U$19.A
- new net N$11: R12.2, U$18.OUT, U$8.G
- new net N$12: CFILTER_1.1, CFILTER_2.1, DCM290P138T600A40.IN+, L_IN.2, R_IN.2
- new net N$13: U$13.S, U$14.D
- new net N$14: D4.A, OK3.EMIT, R17.2
- new net N$15: D1.A, R11.1, U$12.D
- new net N$16: R16.2, U$19.K
- new net N$17: R14.2, U$8.D
- new net N$18: 1A_500V_FUSE_IMD_VSENSE.P$2, U$17.P$2
- new net N$19: 1A_500V_FUSE_ENERGYMETER.P$2, U$17.P$1
- new net N$2: R1.2, U$11.G, U$15.GATE
- new net N$20: R14.1, R15.2, U$20.G, U$21.G, U$22.G
- new net N$21: U$24.P$1, U$4.8
- new net N$22: OK3.A, R16.1
- new net N$23: U$4.4, U$4.6
- new net N$24: IC2.D1, IC2.D2, U$4.0
- new net N$25: U$27.NOB3, U$28.NOA3
- new net N$26: U$28.NOB3, U$29.COIL-, U$30.COIL-
- new net N$3: R3.2, U$12.G
- new net N$4: C2.1, IC1.CON
- new net N$5: IC1.DIS, R10.2, R9.1
- new net N$6: R5.2, U$13.G
- new net N$7: R7.2, U$14.G
- new net N$8: IC1.OUT, R7.1, R8.2
- new net N$9: C1.1, IC1.TRE, IC1.TRI, R10.1
- new net NO1A: U$25.P$9, U$26.P$9, U$29.NOA3
- new net NO1B: U$25.P$10, U$26.P$10, U$29.NOB3
- new net NO2A: U$25.P$11, U$26.P$11, U$29.NOA2
- new net NO2B: U$25.P$12, U$26.P$12, U$29.NOB2
- new net NO3A: U$23.P$1, U$26.P$13, U$29.NOA1
- new net NO3B: U$23.P$2, U$26.P$14, U$29.NOB1
- new net NO4A: U$23.P$3, U$26.P$15, U$30.NOA3
- new net NO4B: U$23.P$4, U$26.P$16, U$30.NOB3
- new net NO5A: U$23.P$5, U$26.P$17, U$30.NOA2
- new net NO5B: U$23.P$6, U$26.P$18, U$30.NOB2
- new net NO6A: U$23.P$7, U$26.P$19, U$30.NOA1
- new net NO6B: U$23.P$8, U$26.P$20, U$30.NOB1
- new net PRECH_ACTIVE: R13.2, U$18.IN-, X1-1.K, X1-2.K
- new net RST1IN: U$25.P$6, U$26.P$6, U$27.NOB2, U$28.COIL+
- new net RST2IN: U$25.P$8, U$26.P$8, U$27.COIL-, U$28.NOA2
- new net SPR1PWR: SPR1.2A, SPR1.2B, U$6.P$3
- new net SPR2PWR: SPR2.2A, SPR2.2B, U$6.P$5
- new net TSAL_GRN_GND: R3.1, R4.2, U$11.D, U$7.P$5
- new net TSAL_RED_GND: U$13.D, U$7.P$4
- new net V+: HV+_FUSE_DRY.P$2, INPUT_FUSE.P$1, U$16.P$1, U$4.2
- new net V+_FUSED: INPUT_FUSE.P$2, L_IN.1, R_IN.1
- new net V-: 1A_500V_FUSE_ENERGYMETER.P$1, 1A_500V_FUSE_IMD_VSENSE.P$1, CFILTER_1.2, CFILTER_2.2, DCM290P138T600A40.IN-, U$16.P$2, U$19.G
Other:
- note added: "+12V GLV MAINS"
- note added: "+12V POWER"
- note added: "ACC LIGHT"
- note added: "Clock to generate 4hz TSAL signal"
- note added: "Current regulators measure current across each AIR PN: IXCY10M90S"
- note added: "DCDC CONVERTER 600W 400 to 13.2V"
- note added: "DCDC INPUT FILTER & FUSE"
- note added: "DCDC OUTPUT"
- note added: "DISCHARGE OUTPUT DISABLE CIRCUIT"
- note added: "DRY POLE SENSE: HV+ DRY TO HV-DRY"
- note added: "E-METER VSENSE"
- note added: "Expansion Relays:"
- note added: "FUSED LV OUTPUTS"
- note added: "HIGH VOLTAGE CIRCUIT"
- note added: "HV CIRCUIT"
- note added: "HV+_DRY"
- note added: "HV-_DRY"
- note added: "IMD VSENSE"
- note added: "IXCY10M90S"
- note added: "If current is detected across AIRs, TSAL is activated."
- note added: "LOW VOLTAGE CIRCUIT"
- note added: "LV Circuit"
- note added: "LV Output Terminals"
- note added: "MAIN 12V OUTPUT"
- note added: "MAINS"
- note added: "Monitor Relays"
- note added: "Mosfet to drive green TSAL LED"
- note added: "Mosfets to drive dashboard troubleshooting LEDs, and Accumulator indicator light"
- note added: "Mosfets to drive red TSAL LED"
- note added: "N Channel mosfet driven by gate driver enables or disables p channel mosfets to allow DCDC to deliver current"
- note added: "R1 - 100 R2 - 1M R3 - 100 R4 - 1M R5 - 100 R6 - 1M R7 - 100 R8 - 1M R9 - 2.2K R10 - 4.7M R11 - 1M R12 - 200 R13 - 200 ------ C1 - 39n C2 - 10n C3 - 100n"
- note added: "Relays For IMD, AMS"
- note added: "TSAL OUTPUT"
- note added: "TSMP OUTPUT"
- note added: "UWO FSAE MOTHERBOARD"
- note added: "UWO FSAE PRECHARGE CIRCUIT"
- note added: "WARN LIGHTS"
- note added: "Zener Diode Vz = 56V: when V > 56V, diode will break down and supply current regulator"
