File: ACC-MB/Rev0/ACC-MB-R0.sch (EAGLE design)
At the start: 82 parts, among them IC1 555, IC2 NUD3124DMT1G, X1 PRECH_IN

Commit message: push
Parts:
- removed H5, H6: MOUNT-HOLE3.3, holes:MOUNT-HOLE3.3
- removed IC2: NUD3124DMT1G, _CUSTOM:SAMACSYS_PARTS_NUD3124DMT1G
- added U$31, U$32: GV224, ACC-MB-R0:GV224
- added U$33: FUSE_HOLDER, ACC-MB-R0:FUSE_HOLDER
- added U$34: G7L, ACC-MB-R0:G7L
- added U$35: TO247RESISTORHEATINK, ACC-MB-R0:TO247RESISTORHEATINK
- 1A_500V_FUSE_ENERGYMETER, 1A_500V_FUSE_IMD_VSENSE, HV+_FUSE_DRY, INPUT_FUSE: device _CUSTOM:_CUSTOM_PARTS_LF_885 -> ACC-MB-R0:_CUSTOM_PARTS_LF_885
- AMS, DISCH, IMD, MONITOR, SPR1, SPR2: device fuse:3568FUSEHOLDER -> ACC-MB-R0:3568FUSEHOLDER
- C1, C2, C3, C4, C5: device resistor:C-USC0805 -> ACC-MB-R0:C-USC0805
- CFILTER_1, CFILTER_2: device _CUSTOM:B58035U5305M062 -> ACC-MB-R0:B58035U5305M062
- COUT_EXT: device resistor:CPOL-USE7.5-16 -> ACC-MB-R0:CPOL-USE7.5-16
- D1, D4: device diode:1N4004 -> ACC-MB-R0:1N4004
- D2: device diode:ZENER-DIODEZD-12.5 -> ACC-MB-R0:ZENER-DIODEZD-12.5
- DCM290P138T600A40: device 111_Custom:VICOR_CHIP_WITH_HEATSINK -> ACC-MB-R0:VICOR_CHIP_WITH_HEATSINK
- H1, H2, H3, H4: device holes:MOUNT-HOLE3.3 -> ACC-MB-R0:MOUNT-HOLE3.3
- IC1: device SparkFun-IC-Special-Function:555P -> ACC-MB-R0:555P
- L_IN: device _CUSTOM:SRP1770TA-390M -> ACC-MB-R0:SRP1770TA-390M
- OK3: device optocoupler:LTV816 -> ACC-MB-R0:LTV816
- R1, R10, R11, R17, R19, R2, R3, R4, R5, R6, R7, R8, R9: device resistor:R-US_R0805 -> ACC-MB-R0:R-US_R0805:1
- R12: device rcl:R-EU_R0805 -> ACC-MB-R0:R-EU_R0805
- R13, R14, R15: device rcl:R-US_R0805 -> ACC-MB-R0:R-US_R0805
- R16: device rcl:R-US_R2010 -> ACC-MB-R0:R-US_R2010
- R_IN: device resistor-power:RMG100-V -> ACC-MB-R0:RMG100-V
- U$1: value PHOENIX_1935789 -> G7L; device _CUSTOM:PHOENIX_1935789 -> ACC-MB-R0:G7L
- U$10, U$11, U$12, U$13, U$14: device transistor-fet:BUZ11 -> ACC-MB-R0:BUZ11
- U$15: device HVIB_v2:MIC4417 -> ACC-MB-R0:MIC4417
- U$16, U$17: device _CUSTOM:DCDC_PARTS_282838-2_TE -> ACC-MB-R0:DCDC_PARTS_282838-2_TE
- U$18: device _CUSTOM:UCC27511AQDBVRQ1 -> ACC-MB-R0:UCC27511AQDBVRQ1
- U$19: device HVIB_v2:_CUSTOM_IXCY10M90SD2PAK -> ACC-MB-R0:_CUSTOM_IXCY10M90SD2PAK
- U$2, U$3: device 111_Custom:HSA25 -> ACC-MB-R0:HSA25
- U$20, U$21, U$22: device PDM_2019_RevB:_CUSTOM_111_CUSTOM_SQJ407EP-T1_GE3 -> ACC-MB-R0:_CUSTOM_111_CUSTOM_SQJ407EP-T1_GE3
- U$23, U$25: device CUSTOM_PARTS:1777642_PHOENIX -> ACC-MB-R0:1777642_PHOENIX
- U$24: value TO247RESISTORHEATINK -> FUSE_HOLDER; device 111:TO247RESISTORHEATINK -> ACC-MB-R0:FUSE_HOLDER
- U$26: device CUSTOM_PARTS:DTM1312PA12BR008 -> ACC-MB-R0:DTM1312PA12BR008
- U$27, U$28, U$29, U$30: device CUSTOM_PARTS:SR4M4012_TE -> ACC-MB-R0:SR4M4012_TE
- U$4: value G7L -> TO247RESISTORHEATINK; device precharge:G7L -> ACC-MB-R0:TO247RESISTORHEATINK
- U$5, U$6: device DCDC_Parts:1935200_PHOENIX -> ACC-MB-R0:1935200_PHOENIX
- U$7: device 111_Custom:PHOENIX_1725724 -> ACC-MB-R0:PHOENIX_1725724
- U$8: device 111_Custom:RK7002BMT116 -> ACC-MB-R0:RK7002BMT116
- U$9: device DCDC_Parts:1777600_PHOENIX -> ACC-MB-R0:1777600_PHOENIX
- X1: device con-phoenix-350:1751248 -> ACC-MB-R0:1751248
Connections:
- removed net CTRL: IC2.G1, IC2.G2, U$1.2
- removed net GNDA: IC2.S1, IC2.S2, U$1.1
- new net HV-_WET: U$32.A2
- new net N$27: U$31.X2, U$32.X1
- new net N$30: U$1.4, U$1.6
- new net N$31: U$1.8, U$4.P$1
- new net SAFETY+: U$31.X1
- new net SAFETY-: U$32.X2
- net +12V: now also U$32.T2; no longer U$1.3, U$4.1
- net GND: now also U$1.0, U$34.0
- net HV+_WET: now also U$31.A1, U$35.P$2; no longer U$24.P$2
- net N$21: now also U$34.8, U$35.P$1; no longer U$24.P$1, U$4.8
- net N$23: now also U$34.4, U$34.6; no longer U$4.4, U$4.6
- net N$24: now also U$1.1, U$32.T1; no longer IC2.D1, IC2.D2, U$4.0
- net V+: now also U$31.A2, U$34.2, U$4.P$2; no longer U$4.2
- net V-: now also U$1.2, U$32.A1
Other:
- note added: "AIR+"
- note added: "AIR-"
- note added: "Discharge Circuit"
- note added: "Precharge Circuit"
- note removed: "+12V GLV MAINS"
- note removed: "HV CIRCUIT"
- note removed: "LV Circuit"
- note removed: "UWO FSAE PRECHARGE CIRCUIT"
