File: ACC-MB/Rev0/ACC-MB-R0.brd (EAGLE design)
At the start: 160 x 100 mm, 82 parts, among them IC1 555, IC2 NUD3124DMT1G, X1 PRECH_IN

Commit message: push
Parts:
- removed H5, H6: MOUNT-HOLE3.3, holes:3,3
- removed IC2: NUD3124DMT1G, _CUSTOM:SAMACSYS_PARTS_SOT95P275X110-6N
- added U$31, U$32: GV224, ACC-MB-R0:GV224
- added U$33: FUSE_HOLDER, ACC-MB-R0:FUSE_HOLDER
- added U$34: G7L, ACC-MB-R0:G7L
- added U$35: TO247RESISTORHEATINK, ACC-MB-R0:_CUSTOM_TO-247-2V
- 1A_500V_FUSE_ENERGYMETER, 1A_500V_FUSE_IMD_VSENSE, HV+_FUSE_DRY, INPUT_FUSE: device _CUSTOM:_CUSTOM_PARTS_LF_885 -> ACC-MB-R0:_CUSTOM_PARTS_LF_885
- AMS, DISCH, IMD, MONITOR, SPR1, SPR2: device fuse:3568 -> ACC-MB-R0:3568
- C1, C2, C3, C4, C5: device resistor:C0805 -> ACC-MB-R0:C0805
- CFILTER_1, CFILTER_2: device _CUSTOM:CERALINK_FA3 -> ACC-MB-R0:CERALINK_FA3
- COUT_EXT: device resistor:E7,5-16 -> ACC-MB-R0:E7,5-16
- D1, D4: device diode:DO41-10 -> ACC-MB-R0:DO41-10
- D2: device diode:ZDIO12.5 -> ACC-MB-R0:ZDIO12.5
- DCM290P138T600A40: device 111_Custom:VICOR_CHIP_HEATSINK -> ACC-MB-R0:VICOR_CHIP_HEATSINK
- H1, H2, H3, H4: device holes:3,3 -> ACC-MB-R0:3,3
- IC1: device SparkFun-IC-Special-Function:DIP08 -> ACC-MB-R0:DIP08
- L_IN: device _CUSTOM:L_1510_NONSTANDARD -> ACC-MB-R0:L_1510_NONSTANDARD
- OK3: device optocoupler:DIL04 -> ACC-MB-R0:DIL04
- R1, R10, R11, R17, R19, R2, R3, R4, R5, R6, R7, R8, R9: device resistor:R0805 -> ACC-MB-R0:R0805:1
- R12, R13, R14, R15: device rcl:R0805 -> ACC-MB-R0:R0805
- R16: device rcl:R2010 -> ACC-MB-R0:R2010
- R_IN: device resistor-power:TO-247-2V -> ACC-MB-R0:TO-247-2V
- U$1: value PHOENIX_1935789 -> G7L; device _CUSTOM:PHOENIX_1935789 -> ACC-MB-R0:G7L
- U$10, U$11, U$12, U$13, U$14: device transistor-fet:TO220 -> ACC-MB-R0:TO220
- U$15: device HVIB_v2:PDM_2019_REVB_MIC4416YM4-TR -> ACC-MB-R0:PDM_2019_REVB_MIC4416YM4-TR
- U$16, U$17: device _CUSTOM:DCDC_PARTS_282838-2_FOOT -> ACC-MB-R0:DCDC_PARTS_282838-2_FOOT
- U$18: device _CUSTOM:SOT23-5L -> ACC-MB-R0:SOT23-5L
- U$19: device HVIB_v2:TO228P991X238-3 -> ACC-MB-R0:TO228P991X238-3
- U$2, U$3: device 111_Custom:HSA_25_FOOT -> ACC-MB-R0:HSA_25_FOOT
- U$20, U$21, U$22: device PDM_2019_RevB:_CUSTOM_111_CUSTOM_TRANS_SIRA90DP-T1-GE3 -> ACC-MB-R0:_CUSTOM_111_CUSTOM_TRANS_SIRA90DP-T1-GE3
- U$23, U$25: device CUSTOM_PARTS:1777642_FOOTPRINT -> ACC-MB-R0:1777642_FOOTPRINT
- U$24: value TO247RESISTORHEATINK -> FUSE_HOLDER; device 111:_CUSTOM_TO-247-2V -> ACC-MB-R0:FUSE_HOLDER
- U$26: device CUSTOM_PARTS:DE_12X2_PIN_HEADER -> ACC-MB-R0:DE_12X2_PIN_HEADER
- U$27, U$28, U$29, U$30: device CUSTOM_PARTS:SR4M4012_FOOT -> ACC-MB-R0:SR4M4012_FOOT
- U$4: value G7L -> TO247RESISTORHEATINK; device precharge:G7L -> ACC-MB-R0:_CUSTOM_TO-247-2V
- U$5, U$6: device DCDC_Parts:1777587_FOOT -> ACC-MB-R0:1777587_FOOT
- U$7: device 111_Custom:1725724_FOOT -> ACC-MB-R0:1725724_FOOT
- U$8: device 111_Custom:SOT23 -> ACC-MB-R0:SOT23
- U$9: device DCDC_Parts:1777600_FOOT -> ACC-MB-R0:1777600_FOOT
- X1: device con-phoenix-350:1751248 -> ACC-MB-R0:1751248
- moved U$1 312.7 mm to (193.0, 11.4), turned to 180 degrees
- moved U$24 309.7 mm to (15.2, 109.2), turned to 90 degrees
- moved U$4 278.7 mm to (125.7, 25.4), turned to 90 degrees
- moved U$2 3.81 mm to (-61.0, 1.27)
Connections:
- removed net CTRL: IC2.2, IC2.5, U$1.2
- removed net GNDA: IC2.1, IC2.4, U$1.1
- new net HV-_WET: U$32.A2
- new net N$27: U$31.X2, U$32.X1
- new net N$30: U$1.4, U$1.6
- new net N$31: U$1.8, U$4.1
- new net SAFETY+: U$31.X1
- new net SAFETY-: U$32.X2
- net +12V: now also U$32.T2; no longer U$1.3, U$4.1
- net GND: now also U$1.0, U$34.0
- net HV+_WET: now also U$31.A1, U$35.2; no longer U$24.2
- net N$21: now also U$34.8, U$35.1; no longer U$24.1, U$4.8
- net N$23: now also U$34.4, U$34.6; no longer U$4.4, U$4.6
- net N$24: now also U$1.1, U$32.T1; no longer IC2.3, IC2.6, U$4.0
- net V+: now also U$31.A2, U$34.2
- net V-: now also U$1.2, U$32.A1
Routing:
- net N$27: track 0.00 -> 206.8 mm
- net GND: track 0.00 -> 174.8 mm
- net N$24: track 0.00 -> 146.5 mm
- net V+: track 0.00 -> 125.0 mm
- net HV+_WET: track 0.00 -> 51.3 mm
- net N$21: track 0.00 -> 47.2 mm
- net V-: track 0.00 -> 37.5 mm
- net N$31: track 0.00 -> 32.3 mm
- net N$30: track 0.00 -> 14.4 mm
- net N$23: track 0.00 -> 14.4 mm
Other:
- board size 160 x 100 mm -> 210.8 x 166 mm
