File: 2019/HOLDUP.brd (EAGLE design)
At the start: 210 x 180 mm, 22 parts

Commit message: brd
Parts:
- removed C2: 15000u, 111_Custom:CAPPRD750W65D1800H3700B
- removed D2: 10A, 111_Custom:DIOAD1570W120L850D500B
- removed H1, H2, H3, H4: MOUNT-HOLE5.5, ACC-MB-R0:5,5
- removed R2: 100, 111_Custom:RESAD976W63L650D250B
- removed U$1, U$2: FUSE_HOLDER, ACC-MB-R0:FUSE_HOLDER
- removed U$10, U$11, U$12, U$3, U$4, U$5, U$6, U$7, U$8, U$9: PCIE-36-CONN, ACC-MB-R0:PCI-E-36-CONN
- added J1: TE_282834-4, 111_Custom:282834-4_FOOT
- moved C1 112.6 mm to (40.0, 9.00), turned to 180 degrees
- moved R1 110.9 mm to (25.0, 3.00)
- moved D1 94.3 mm to (10.0, 15.0)
Connections:
- removed net +12V: U$7.B1, U$7.B10, U$7.B11, U$7.B12, U$7.B13, U$7.B14, U$7.B15, U$7.B16, U$7.B17, U$7.B18, U$7.B2, U$7.B3, U$7.B4, U$7.B5, U$7.B6, U$7.B7, U$7.B8, U$7.B9
- removed net GND: U$7.A1, U$7.A10, U$7.A11, U$7.A12, U$7.A13, U$7.A14, U$7.A15, U$7.A16, U$7.A17, U$7.A18, U$7.A2, U$7.A3, U$7.A4, U$7.A5, U$7.A6, U$7.A7, U$7.A8, U$7.A9
- removed net N$4: D2.1, R2.1
- removed net N$5: C2.2
- removed net N$6: C2.1, D2.2, R2.2
- net N$1: now also J1.P$2, J1.P$4
- net N$2: now also J1.P$1, J1.P$3
Routing:
- net N$3: track 0.00 -> 45.5 mm
- net N$2: track 0.00 -> 42.4 mm
- net N$1: track 0.00 -> 32.2 mm
Other:
- board size 210 x 180 mm -> 49.2 x 28 mm
- board text added: "+IN"
- board text added: "+OUT"
- board text added: "-IN"
- board text added: "-OUT"
- board text removed: "AIR+"
- board text removed: "AIR-"
- board text removed: "DCDC"
- board text removed: "Discharge"
- board text removed: "Main Fuse"
- board text removed: "Precharge"
