File: ACC-MB/Rev0/CRDC/CRDC.sch (EAGLE design)
At the start: 5 parts

Commit message: update
Parts:
- removed U$4: IPBT-102-H1-T-D, ACC-MB-R0:IPBT-102-H1-T-D
- added X5: 5566-8, con-molex:5566-8
Connections:
- net HV+_WET: now also X5-3.S, X5-4.S, X5-7.S, X5-8.S; no longer U$4.P$3, U$4.P$4
- net V+: now also X5-1.S, X5-2.S, X5-5.S, X5-6.S; no longer U$4.P$1, U$4.P$2
Changed lines of the file:
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@@
 <part name="FRAME3" library="ACC-MB-R0" deviceset="A3L-LOC" device=""/>
 <part name="U$1" library="ACC-MB-R0" library_urn="urn:adsk.eagle:library:13324935" deviceset="G7L" device="" package3d_urn="urn:adsk.eagle:package:13209535/2"/>
-<part name="U$4" library="ACC-MB-R0" library_urn="urn:adsk.eagle:library:13324935" deviceset="IPBT-102-H1-T-D" device="" package3d_urn="urn:adsk.eagle:package:13324986/2"/>
 <part name="U$5" library="ACC-MB-R0" library_urn="urn:adsk.eagle:library:13324935" deviceset="TO247RESISTORHEATINK" device="" package3d_urn="urn:adsk.eagle:package:13209502/3"/>
 <part name="U$2" library="ACC-MB-R0" library_urn="urn:adsk.eagle:library:13324935" deviceset="PCIE-36-EDGE" device=""/>
 <part name="U$3" library="ACC-MB-R0" library_urn="urn:adsk.eagle:library:13324935" deviceset="PCIE-36-EDGE" device=""/>
+<part name="X5" library="con-molex" library_urn="urn:adsk.eagle:library:165" deviceset="5566-8" device=""/>
 </parts>
 <sheets>
@@
 </instance>
 <instance part="U$1" gate="G$1" x="119.38" y="172.72" rot="R180"/>
-<instance part="U$4" gate="G$1" x="109.22" y="203.2" rot="R180"/>
 <instance part="U$5" gate="G$1" x="88.9" y="180.34" rot="R180"/>
 <instance part="U$2" gate="G$1" x="111.76" y="154.94"/>
 <instance part="U$3" gate="G$1" x="149.86" y="154.94"/>
+<instance part="X5" gate="-1" x="157.48" y="208.28"/>
+<instance part="X5" gate="-2" x="157.48" y="205.74"/>
+<instance part="X5" gate="-3" x="157.48" y="203.2"/>
+<instance part="X5" gate="-4" x="157.48" y="200.66"/>
+<instance part="X5" gate="-5" x="157.48" y="198.12"/>
+<instance part="X5" gate="-6" x="157.48" y="195.58"/>
+<instance part="X5" gate="-7" x="157.48" y="193.04"/>
+<instance part="X5" gate="-8" x="157.48" y="190.5"/>
 </instances>
 <busses>
@@
 <segment>
 <wire x1="71.12" y1="180.34" x2="76.2" y2="180.34" width="0.1524" layer="91"/>
-<wire x1="83.82" y1="198.12" x2="96.52" y2="198.12" width="0.1524" layer="91"/>
-<wire x1="96.52" y1="203.2" x2="83.82" y2="203.2" width="0.1524" layer="91"/>
-<wire x1="83.82" y1="203.2" x2="83.82" y2="198.12" width="0.1524" layer="91"/>
 <wire x1="71.12" y1="180.34" x2="71.12" y2="198.12" width="0.1524" layer="91"/>
-<wire x1="71.12" y1="198.12" x2="83.82" y2="198.12" width="0.1524" layer="91"/>
-<junction x="83.82" y="198.12"/>
-<pinref part="U$4" gate="G$1" pin="P$3"/>
-<pinref part="U$4" gate="G$1" pin="P$4"/>
+<wire x1="71.12" y1="198.12" x2="96.52" y2="198.12" width="0.1524" layer="91"/>
 <pinref part="U$5" gate="G$1" pin="P$2"/>
+<pinref part="X5" gate="-4" pin="S"/>
+<wire x1="154.94" y1="200.66" x2="152.4" y2="200.66" width="0.1524" layer="91"/>
+<wire x1="152.4" y1="200.66" x2="96.52" y2="200.66" width="0.1524" layer="91"/>
+<wire x1="96.52" y1="200.66" x2="96.52" y2="198.12" width="0.1524" layer="91"/>
+<pinref part="X5" gate="-3" pin="S"/>
+<wire x1="154.94" y1="203.2" x2="152.4" y2="203.2" width="0.1524" layer="91"/>
+<wire x1="152.4" y1="203.2" x2="152.4" y2="200.66" width="0.1524" layer="91"/>
+<junction x="152.4" y="200.66"/>
+<pinref part="X5" gate="-7" pin="S"/>
+<wire x1="152.4" y1="200.66" x2="152.4" y2="193.04" width="0.1524" layer="91"/>
+<wire x1="152.4" y1="193.04" x2="154.94" y2="193.04" width="0.1524" layer="91"/>
+<pinref part="X5" gate="-8" pin="S"/>
+<wire x1="152.4" y1="193.04" x2="152.4" y2="190.5" width="0.1524" layer="91"/>
+<wire x1="152.4" y1="190.5" x2="154.94" y2="190.5" width="0.1524" layer="91"/>
+<junction x="152.4" y="193.04"/>
 </segment>
 </net>
@@
 <net name="V+" class="1">
 <segment>
-<wire x1="132.08" y1="172.72" x2="154.94" y2="172.72" width="0.1524" layer="91"/>
-<wire x1="119.38" y1="198.12" x2="132.08" y2="198.12" width="0.1524" layer="91"/>
-<wire x1="119.38" y1="203.2" x2="132.08" y2="203.2" width="0.1524" layer="91"/>
-<wire x1="132.08" y1="203.2" x2="132.08" y2="198.12" width="0.1524" layer="91"/>
-<wire x1="154.94" y1="172.72" x2="154.94" y2="198.12" width="0.1524" layer="91"/>
-<wire x1="154.94" y1="198.12" x2="132.08" y2="198.12" width="0.1524" layer="91"/>
-<junction x="132.08" y="198.12"/>
+<wire x1="132.08" y1="172.72" x2="149.86" y2="172.72" width="0.1524" layer="91"/>
 <pinref part="U$1" gate="G$1" pin="2"/>
-<pinref part="U$4" gate="G$1" pin="P$1"/>
-<pinref part="U$4" gate="G$1" pin="P$2"/>
+<pinref part="X5" gate="-5" pin="S"/>
+<wire x1="154.94" y1="195.58" x2="154.94" y2="198.12" width="0.1524" layer="91"/>
+<pinref part="X5" gate="-6" pin="S"/>
+<wire x1="154.94" y1="195.58" x2="149.86" y2="195.58" width="0.1524" layer="91"/>
+<junction x="154.94" y="195.58"/>
+<wire x1="149.86" y1="195.58" x2="149.86" y2="172.72" width="0.1524" layer="91"/>
+<wire x1="149.86" y1="195.58" x2="149.86" y2="205.74" width="0.1524" layer="91"/>
+<junction x="149.86" y="195.58"/>
+<pinref part="X5" gate="-2" pin="S"/>
+<wire x1="149.86" y1="205.74" x2="152.4" y2="205.74" width="0.1524" layer="91"/>
+<pinref part="X5" gate="-1" pin="S"/>
+<wire x1="152.4" y1="205.74" x2="154.94" y2="205.74" width="0.1524" layer="91"/>
+<wire x1="154.94" y1="208.28" x2="152.4" y2="208.28" width="0.1524" layer="91"/>
+<wire x1="152.4" y1="208.28" x2="152.4" y2="205.74" width="0.1524" layer="91"/>
+<junction x="152.4" y="205.74"/>
 </segment>
 </net>
