File: ACC-MB/Rev0/DCDCDC/DCDCDC.sch (EAGLE design)
At the start: 20 parts

Commit message: update
Parts:
- removed U$8: IPBT-102-H1-T-D, ACC-MB-R0:IPBT-102-H1-T-D
- added X5: 5566-8, con-molex:5566-8
Connections:
- net V+: now also X5-1.S, X5-2.S, X5-5.S; no longer U$8.P$1, U$8.P$2
- net V-: now also X5-4.S, X5-7.S, X5-8.S; no longer U$8.P$3, U$8.P$4
Changed lines of the file:
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@@
 </variantdefs>
 <classes>
-<class number="0" name="LOW" width="0" drill="0">
+<class number="0" name="default" width="1" drill="0">
 <clearance class="0" value="0.1524"/>
 </class>
-<class number="1" name="HV" width="1" drill="0">
-<clearance class="1" value="2"/>
+<class number="1" name="LV" width="0" drill="0">
+<clearance class="1" value="0.0005"/>
 </class>
 </classes>
@@
 <part name="U$6" library="PDM_2019_RevB" deviceset="_CUSTOM_111_CUSTOM_SQJ407EP-T1_GE3" device=""/>
 <part name="U$3" library="PDM_2019_RevB" deviceset="_CUSTOM_111_CUSTOM_SQJ407EP-T1_GE3" device=""/>
-<part name="U$8" library="ACC-MB-R0" library_urn="urn:adsk.eagle:library:13324935" deviceset="IPBT-102-H1-T-D" device="" package3d_urn="urn:adsk.eagle:package:13324986/2"/>
 <part name="U$10" library="ACC-MB-R0" library_urn="urn:adsk.eagle:library:13324935" deviceset="PCIE-36-EDGE" device=""/>
 <part name="U$1" library="ACC-MB-R0" library_urn="urn:adsk.eagle:library:13324935" deviceset="IPBT-102-H1-T-D" device="" package3d_urn="urn:adsk.eagle:package:13324986/2"/>
@@
 <part name="P+6" library="supply1" library_urn="urn:adsk.eagle:library:371" deviceset="+12V" device=""/>
 <part name="U$2" library="ACC-MB-R0" library_urn="urn:adsk.eagle:library:13324935" deviceset="PCIE-36-EDGE" device=""/>
+<part name="P+7" library="ACC-MB-R0" deviceset="V+" device=""/>
+<part name="P-5" library="ACC-MB-R0" deviceset="V-" device=""/>
+<part name="X5" library="con-molex" library_urn="urn:adsk.eagle:library:165" deviceset="5566-8" device=""/>
 </parts>
 <sheets>
@@
 <instance part="U$6" gate="G$1" x="256.54" y="213.36"/>
 <instance part="U$3" gate="G$1" x="256.54" y="228.6"/>
-<instance part="U$8" gate="G$1" x="30.48" y="209.55" rot="R270"/>
 <instance part="U$10" gate="G$1" x="346.71" y="88.9"/>
 <instance part="U$1" gate="G$1" x="314.96" y="57.15"/>
@@
 </instance>
 <instance part="U$2" gate="G$1" x="190.5" y="139.7"/>
+<instance part="P+7" gate="1" x="57.15" y="152.4" smashed="yes">
+<attribute name="VALUE" x="54.61" y="149.86" size="1.778" layer="96" rot="R90"/>
+</instance>
+<instance part="P-5" gate="1" x="54.61" y="127" smashed="yes">
+<attribute name="VALUE" x="49.53" y="129.54" size="1.778" layer="96" rot="R270"/>
+</instance>
+<instance part="X5" gate="-1" x="62.23" y="148.59"/>
+<instance part="X5" gate="-2" x="62.23" y="146.05"/>
+<instance part="X5" gate="-3" x="62.23" y="143.51"/>
+<instance part="X5" gate="-4" x="62.23" y="140.97"/>
+<instance part="X5" gate="-5" x="62.23" y="138.43"/>
+<instance part="X5" gate="-6" x="62.23" y="135.89"/>
+<instance part="X5" gate="-7" x="62.23" y="133.35"/>
+<instance part="X5" gate="-8" x="62.23" y="130.81"/>
 </instances>
 <busses>
@@
 <wire x1="27.94" y1="219.71" x2="27.94" y2="227.33" width="0.1524" layer="91"/>
 <pinref part="INPUT_FUSE" gate="G$1" pin="P$1"/>
-<wire x1="36.83" y1="219.71" x2="35.56" y2="219.71" width="0.1524" layer="91"/>
-<wire x1="35.56" y1="219.71" x2="30.48" y2="219.71" width="0.1524" layer="91"/>
-<pinref part="U$8" gate="G$1" pin="P$1"/>
-<junction x="35.56" y="219.71"/>
-<pinref part="U$8" gate="G$1" pin="P$2"/>
-<wire x1="30.48" y1="219.71" x2="27.94" y2="219.71" width="0.1524" layer="91"/>
-<junction x="30.48" y="219.71"/>
+<wire x1="36.83" y1="219.71" x2="27.94" y2="219.71" width="0.1524" layer="91"/>
+</segment>
+<segment>
+<pinref part="P+7" gate="1" pin="V+"/>
+<pinref part="X5" gate="-1" pin="S"/>
+<wire x1="57.15" y1="148.59" x2="57.15" y2="149.86" width="0.1524" layer="91"/>
+<wire x1="59.69" y1="148.59" x2="57.15" y2="148.59" width="0.1524" layer="91"/>
+<junction x="57.15" y="148.59"/>
+<pinref part="X5" gate="-5" pin="S"/>
+<wire x1="57.15" y1="148.59" x2="57.15" y2="146.05" width="0.1524" layer="91"/>
+<wire x1="57.15" y1="146.05" x2="57.15" y2="138.43" width="0.1524" layer="91"/>
+<wire x1="57.15" y1="138.43" x2="59.69" y2="138.43" width="0.1524" layer="91"/>
+<pinref part="X5" gate="-2" pin="S"/>
+<wire x1="59.69" y1="146.05" x2="57.15" y2="146.05" width="0.1524" layer="91"/>
+<junction x="57.15" y="146.05"/>
 </segment>
 </net>
@@
 <pinref part="P-1" gate="1" pin="V-"/>
 <wire x1="27.94" y1="196.85" x2="27.94" y2="181.61" width="0.1524" layer="91"/>
-<wire x1="27.94" y1="196.85" x2="30.48" y2="196.85" width="0.1524" layer="91"/>
 <pinref part="CFILTER_1" gate="G$1" pin="2"/>
-<wire x1="30.48" y1="196.85" x2="35.56" y2="196.85" width="0.1524" layer="91"/>
-<wire x1="35.56" y1="196.85" x2="86.36" y2="196.85" width="0.1524" layer="91"/>
+<wire x1="27.94" y1="196.85" x2="86.36" y2="196.85" width="0.1524" layer="91"/>
 <wire x1="86.36" y1="196.85" x2="95.25" y2="196.85" width="0.1524" layer="91"/>
 <wire x1="86.36" y1="209.55" x2="86.36" y2="196.85" width="0.1524" layer="91"/>
@@
 <wire x1="99.06" y1="196.85" x2="95.25" y2="196.85" width="0.1524" layer="91"/>
 <junction x="95.25" y="196.85"/>
-<pinref part="U$8" gate="G$1" pin="P$3"/>
-<junction x="30.48" y="196.85"/>
-<pinref part="U$8" gate="G$1" pin="P$4"/>
-<junction x="35.56" y="196.85"/>
+</segment>
+<segment>
+<pinref part="X5" gate="-8" pin="S"/>
+<wire x1="54.61" y1="130.81" x2="59.69" y2="130.81" width="0.1524" layer="91"/>
+<pinref part="P-5" gate="1" pin="V-"/>
+<wire x1="54.61" y1="129.54" x2="54.61" y2="130.81" width="0.1524" layer="91"/>
+<junction x="54.61" y="130.81"/>
+<pinref part="X5" gate="-4" pin="S"/>
+<wire x1="59.69" y1="140.97" x2="54.61" y2="140.97" width="0.1524" layer="91"/>
+<wire x1="54.61" y1="140.97" x2="54.61" y2="133.35" width="0.1524" layer="91"/>
+<pinref part="X5" gate="-7" pin="S"/>
+<wire x1="54.61" y1="133.35" x2="54.61" y2="130.81" width="0.1524" layer="91"/>
+<wire x1="59.69" y1="133.35" x2="54.61" y2="133.35" width="0.1524" layer="91"/>
+<junction x="54.61" y="133.35"/>
 </segment>
 </net>

Commit message: update
Parts:
- removed U$1: IPBT-102-H1-T-D, ACC-MB-R0:IPBT-102-H1-T-D
- added X1: 5566-8, con-molex:5566-8
Connections:
- new net N$5: X1-1.S, X1-2.S, X1-5.S
- new net N$6: X1-4.S, X1-7.S, X1-8.S
- net +12V: no longer U$1.P$1, U$1.P$2
- net GND: no longer U$1.P$3, U$1.P$4
Changed lines of the file:
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@@
 <part name="R1" library="rcl" library_urn="urn:adsk.eagle:library:334" deviceset="R-EU_" device="R0805" package3d_urn="urn:adsk.eagle:package:23553/2"/>
 <part name="GND3" library="supply1" library_urn="urn:adsk.eagle:library:371" deviceset="GND" device=""/>
-<part name="GND5" library="supply1" library_urn="urn:adsk.eagle:library:371" deviceset="GND" device=""/>
-<part name="P+4" library="supply1" library_urn="urn:adsk.eagle:library:371" deviceset="+12V" device=""/>
 <part name="U$5" library="_CUSTOM" deviceset="UCC27511AQDBVRQ1" device=""/>
 <part name="R2" library="rcl" library_urn="urn:adsk.eagle:library:334" deviceset="R-US_" device="R0805" package3d_urn="urn:adsk.eagle:package:23553/2"/>
@@
 <part name="U$3" library="PDM_2019_RevB" deviceset="_CUSTOM_111_CUSTOM_SQJ407EP-T1_GE3" device=""/>
 <part name="U$10" library="ACC-MB-R0" library_urn="urn:adsk.eagle:library:13324935" deviceset="PCIE-36-EDGE" device=""/>
-<part name="U$1" library="ACC-MB-R0" library_urn="urn:adsk.eagle:library:13324935" deviceset="IPBT-102-H1-T-D" device="" package3d_urn="urn:adsk.eagle:package:13324986/2"/>
 <part name="GND7" library="supply1" library_urn="urn:adsk.eagle:library:371" deviceset="GND" device=""/>
 <part name="P+6" library="supply1" library_urn="urn:adsk.eagle:library:371" deviceset="+12V" device=""/>
 <part name="U$2" library="ACC-MB-R0" library_urn="urn:adsk.eagle:library:13324935" deviceset="PCIE-36-EDGE" device=""/>
-<part name="P+7" library="ACC-MB-R0" deviceset="V+" device=""/>
-<part name="P-5" library="ACC-MB-R0" deviceset="V-" device=""/>
+<part name="P+7" library="ACC-MB-R0" library_urn="urn:adsk.eagle:library:13208985" deviceset="V+" device=""/>
+<part name="P-5" library="ACC-MB-R0" library_urn="urn:adsk.eagle:library:13208985" deviceset="V-" device=""/>
 <part name="X5" library="con-molex" library_urn="urn:adsk.eagle:library:165" deviceset="5566-8" device=""/>
+<part name="X1" library="con-molex" library_urn="urn:adsk.eagle:library:165" deviceset="5566-8" device=""/>
+<part name="P+5" library="supply1" library_urn="urn:adsk.eagle:library:371" deviceset="+12V" device=""/>
+<part name="GND1" library="supply1" library_urn="urn:adsk.eagle:library:371" deviceset="GND" device=""/>
 </parts>
 <sheets>
@@
 <attribute name="VALUE" x="283.21" y="161.29" size="1.778" layer="96"/>
 </instance>
-<instance part="GND5" gate="1" x="332.74" y="50.8" smashed="yes">
-<attribute name="VALUE" x="330.2" y="48.26" size="1.778" layer="96"/>
-</instance>
-<instance part="P+4" gate="1" x="299.72" y="73.66" smashed="yes">
-<attribute name="VALUE" x="297.18" y="68.58" size="1.778" layer="96" rot="R90"/>
-</instance>
 <instance part="U$5" gate="G$1" x="207.01" y="226.06"/>
 <instance part="R2" gate="G$1" x="234.95" y="173.99" rot="R90"/>
@@
 <instance part="U$3" gate="G$1" x="256.54" y="228.6"/>
 <instance part="U$10" gate="G$1" x="346.71" y="88.9"/>
-<instance part="U$1" gate="G$1" x="314.96" y="57.15"/>
 <instance part="GND7" gate="1" x="340.36" y="35.56" smashed="yes">
 <attribute name="VALUE" x="337.82" y="33.02" size="1.778" layer="96"/>
@@
 <instance part="X5" gate="-7" x="62.23" y="133.35"/>
 <instance part="X5" gate="-8" x="62.23" y="130.81"/>
+<instance part="X1" gate="-1" x="317.5" y="66.04"/>
+<instance part="X1" gate="-2" x="317.5" y="63.5"/>
+<instance part="X1" gate="-3" x="317.5" y="60.96"/>
+<instance part="X1" gate="-4" x="317.5" y="58.42"/>
+<instance part="X1" gate="-5" x="317.5" y="55.88"/>
+<instance part="X1" gate="-6" x="317.5" y="53.34"/>
+<instance part="X1" gate="-7" x="317.5" y="50.8"/>
+<instance part="X1" gate="-8" x="317.5" y="48.26"/>
+<instance part="P+5" gate="1" x="312.42" y="78.74" smashed="yes">
+<attribute name="VALUE" x="309.88" y="73.66" size="1.778" layer="96" rot="R90"/>
+</instance>
+<instance part="GND1" gate="1" x="309.88" y="40.64" smashed="yes">
+<attribute name="VALUE" x="307.34" y="38.1" size="1.778" layer="96"/>
+</instance>
 </instances>
 <busses>
@@
 <wire x1="162.56" y1="195.58" x2="143.51" y2="195.58" width="0.1524" layer="91"/>
 <junction x="143.51" y="195.58"/>
-</segment>
-<segment>
-<pinref part="U$1" gate="G$1" pin="P$4"/>
-<wire x1="327.66" y1="62.23" x2="332.74" y2="62.23" width="0.1524" layer="91"/>
-<pinref part="GND5" gate="1" pin="GND"/>
-<wire x1="332.74" y1="62.23" x2="332.74" y2="57.15" width="0.1524" layer="91"/>
-<pinref part="U$1" gate="G$1" pin="P$3"/>
-<wire x1="332.74" y1="57.15" x2="332.74" y2="53.34" width="0.1524" layer="91"/>
-<wire x1="327.66" y1="57.15" x2="332.74" y2="57.15" width="0.1524" layer="91"/>
-<junction x="332.74" y="57.15"/>
 </segment>
 <segment>
@@
 <wire x1="340.36" y1="43.18" x2="340.36" y2="40.64" width="0.1524" layer="91"/>
 </segment>
+<segment>
+<pinref part="GND1" gate="1" pin="GND"/>
+<wire x1="309.88" y1="46.99" x2="309.88" y2="43.18" width="0.1524" layer="91"/>
+</segment>
 </net>
 <net name="V+" class="1">
@@
 <wire x1="194.31" y1="220.98" x2="194.31" y2="231.14" width="0.1524" layer="91"/>
 <junction x="194.31" y="231.14"/>
-</segment>
-<segment>
-<pinref part="P+4" gate="1" pin="+12V"/>
-<pinref part="U$1" gate="G$1" pin="P$2"/>
-<wire x1="299.72" y1="71.12" x2="299.72" y2="62.23" width="0.1524" layer="91"/>
-<wire x1="299.72" y1="62.23" x2="299.72" y2="57.15" width="0.1524" layer="91"/>
-<wire x1="299.72" y1="57.15" x2="304.8" y2="57.15" width="0.1524" layer="91"/>
-<pinref part="U$1" gate="G$1" pin="P$1"/>
-<wire x1="304.8" y1="62.23" x2="299.72" y2="62.23" width="0.1524" layer="91"/>
-<junction x="299.72" y="62.23"/>
 </segment>
 <segment>
@@
 <junction x="367.03" y="63.5"/>
 </segment>
+<segment>
+<pinref part="P+5" gate="1" pin="+12V"/>
+<wire x1="312.42" y1="76.2" x2="312.42" y2="67.31" width="0.1524" layer="91"/>
+</segment>
 </net>
 <net name="N$2" class="0">
@@
 </segment>
 </net>
+<net name="N$5" class="1">
+<segment>
+<pinref part="X1" gate="-1" pin="S"/>
+<wire x1="312.42" y1="66.04" x2="312.42" y2="67.31" width="0.1524" layer="91"/>
+<wire x1="314.96" y1="66.04" x2="312.42" y2="66.04" width="0.1524" layer="91"/>
+<junction x="312.42" y="66.04"/>
+<pinref part="X1" gate="-5" pin="S"/>
+<wire x1="312.42" y1="66.04" x2="312.42" y2="63.5" width="0.1524" layer="91"/>
+<wire x1="312.42" y1="63.5" x2="312.42" y2="55.88" width="0.1524" layer="91"/>
+<wire x1="312.42" y1="55.88" x2="314.96" y2="55.88" width="0.1524" layer="91"/>
+<pinref part="X1" gate="-2" pin="S"/>
+<wire x1="314.96" y1="63.5" x2="312.42" y2="63.5" width="0.1524" layer="91"/>
+<junction x="312.42" y="63.5"/>
+</segment>
+</net>
+<net name="N$6" class="1">
+<segment>
+<pinref part="X1" gate="-8" pin="S"/>
+<wire x1="309.88" y1="48.26" x2="314.96" y2="48.26" width="0.1524" layer="91"/>
+<wire x1="309.88" y1="46.99" x2="309.88" y2="48.26" width="0.1524" layer="91"/>
+<junction x="309.88" y="48.26"/>
+<pinref part="X1" gate="-4" pin="S"/>
+<wire x1="314.96" y1="58.42" x2="309.88" y2="58.42" width="0.1524" layer="91"/>
+<wire x1="309.88" y1="58.42" x2="309.88" y2="50.8" width="0.1524" layer="91"/>
+<pinref part="X1" gate="-7" pin="S"/>
+<wire x1="309.88" y1="50.8" x2="309.88" y2="48.26" width="0.1524" layer="91"/>
+<wire x1="314.96" y1="50.8" x2="309.88" y2="50.8" width="0.1524" layer="91"/>
+<junction x="309.88" y="50.8"/>
+</segment>
+</net>
