File: ACC-MB/Rev0/MainBoard/Main.brd (EAGLE design)
At the start: 210 x 180 mm, 61 parts, among them IC1 555, X2 5566-8, X3 5566-8, X5 5566-8

Commit message: model
Parts:
- removed X2, X3: 5566-8, con-molex:5566-8
- added U$13, U$14: SR4M4012_TE, Main:SR4M4012_FOOT
- added X1: 5566-24, Main:5566-24
- 1A_500V_FUSE_ENERGYMETER, 1A_500V_FUSE_IMD_VSENSE, HV+_FUSE_DRY: device ACC-MB-R0:_CUSTOM_PARTS_LF_885 -> Main:_CUSTOM_PARTS_LF_885
- C1, C2: device 111_Custom:CAPPRD750W65D1800H3700B -> Main:CAPPRD750W65D1800H3700B
- C3, C4, C5, C6, C7: device ACC-MB-R0:C0805 -> Main:C0805
- D1, D2: device 111_Custom:DIOAD1570W120L850D500B -> Main:DIOAD1570W120L850D500B
- D3, D4: device ACC-MB-R0:DO41-10 -> Main:DO41-10
- D5: device ACC-MB-R0:ZDIO12.5 -> Main:ZDIO12.5
- H1, H2, H3, H4: device ACC-MB-R0:5,5 -> Main:5,5
- IC1: device ACC-MB-R0:DIP08 -> Main:DIP08
- OK3: device ACC-MB-R0:DIL04 -> Main:DIL04
- R1, R2: device 111_Custom:RESAD976W63L650D250B -> Main:RESAD976W63L650D250B
- R16: device ACC-MB-R0:R2010 -> Main:R2010
- U$1, U$2: device ACC-MB-R0:FUSE_HOLDER -> Main:FUSE_HOLDER
- U$10, U$11, U$12, U$3, U$4, U$5, U$6, U$7, U$8, U$9: device ACC-MB-R0:PCI-E-36-CONN -> Main:PCI-E-36-CONN
- U$15, U$16, U$17, U$18, U$19: device ACC-MB-R0:TO220 -> Main:TO220
- U$22: device ACC-MB-R0:TO228P991X238-3 -> Main:TO228P991X238-3
- U$23: device ACC-MB-R0:PDM_2019_REVB_MIC4416YM4-TR -> Main:PDM_2019_REVB_MIC4416YM4-TR
- U$24, U$25: device ACC-MB-R0:HSA_25_FOOT -> Main:HSA_25_FOOT
- X5: device con-molex:5566-8 -> Main:5566-8
- moved U$25 368.2 mm to (251.0, 98.0), turned to 90 degrees
Connections:
- removed net N$23: D1.1, R1.1, U$4.B1, U$4.B10, U$4.B11, U$4.B2, U$4.B3, U$4.B4, U$4.B5, U$4.B6, U$4.B7, U$4.B8, U$4.B9, X3.5, X3.6, X3.7, X3.8
- new net CH1IN: U$13.NOA2
- new net CH2IN: U$14.NOB2
- new net N$19: U$14.NOB3
- new net PRECHARGE+: U$9.A1, U$9.A10, U$9.A11, U$9.A12, U$9.A13, U$9.A14, U$9.A15, U$9.A16, U$9.A17, U$9.A18, U$9.A2, U$9.A3, U$9.A4, U$9.A5, U$9.A6, U$9.A7, U$9.A8, U$9.A9, X1.14
- new net RST1IN: U$13.NOB2, U$14.COIL+
- new net RST2IN: U$13.COIL-, U$14.NOA2
- new net SAFETY+: D1.1, R1.1, U$4.B1, U$4.B10, U$4.B11, U$4.B2, U$4.B3, U$4.B4, U$4.B5, U$4.B6, U$4.B7, U$4.B8, U$4.B9, X1.1
- new net SAFETY-: C2.2, U$5.B12, U$5.B13, U$5.B14, U$5.B15, U$5.B16, U$5.B17, U$5.B18, X1.13
- net +12V: now also U$13.NOA3; no longer X2.2, X2.4, X2.8
- net ACC_LGHT: now also X1.11; no longer X2.7
- net GND: now also U$13.COIL+, U$14.COIL-, U$9.B1, U$9.B10, U$9.B11, U$9.B12, U$9.B13, U$9.B14, U$9.B15, U$9.B16, U$9.B17, U$9.B18, U$9.B2, U$9.B3, U$9.B4, U$9.B5, U$9.B6, U$9.B7, U$9.B8, U$9.B9, X1.2, X1.24; no longer X2.1, X2.3
- net N$5: now also U$13.NOB3, U$14.NOA3; no longer C2.2, U$5.B12, U$5.B13, U$5.B14, U$5.B15, U$5.B16, U$5.B17, U$5.B18, X3.1, X3.2, X3.3, X3.4
- net TSAL_GRN_GND: now also X1.10; no longer X2.6
- net TSAL_RED_GND: now also X1.12; no longer X2.5
Routing:
- net SAFETY-: track 0.00 -> 285.4 mm
- net PRECHARGE+: track 0.00 -> 283.7 mm
- net N$5: track 268.6 -> 0.00 mm
- net N$23: track 119.0 -> 0.00 mm
- net TSAL_RED_GND: track 67.7 -> 169.5 mm
- net SAFETY+: track 0.00 -> 87.9 mm
- net ACC_LGHT: track 69.8 -> 150.1 mm
- net TSAL_GRN_GND: track 96.8 -> 155.1 mm
- net DISCHARGE+: track 224.2 -> 247.6 mm
- net N$4: track 248.1 -> 235.0 mm

Commit message: update
Parts:
- moved U$4 36.1 mm to (33.0, 29.8), turned to 90 degrees
- moved U$3 35.9 mm to (32.0, 79.8), turned to 90 degrees
- moved U$24 20.0 mm to (-108.0, -15.0)
- moved C1 19.1 mm to (19.0, 17.0), turned to 0 degrees
- moved R1 13.6 mm to (9.00, 32.0)
- moved D1 12.2 mm to (17.0, 33.0)
Routing:
- net SAFETY-: track 285.4 -> 176.7 mm
- net N$4: track 235.0 -> 148.3 mm
- net SAFETY+: track 87.9 -> 15.6 mm
- net DISCHARGE+: track 247.6 -> 213.6 mm
- net N$3: track 25.7 -> 0.00 mm
- net N$6: track 18.7 -> 0.00 mm
