File: ACC-MB/Rev0/MainBoard/Main.sch (EAGLE design)
At the start: 22 parts

Commit message: main
Parts:
- added 1A_500V_FUSE_ENERGYMETER, 1A_500V_FUSE_IMD_VSENSE, HV+_FUSE_DRY: _CUSTOM_PARTS_LF_885, ACC-MB-R0:_CUSTOM_PARTS_LF_885
- added C3: 39n, ACC-MB-R0:C-USC0805
- added C4: 10n, ACC-MB-R0:C-USC0805
- added C5: 100n, ACC-MB-R0:C-USC0805
- added C6: 4.7u, ACC-MB-R0:C-USC0805
- added C7: 0.1u, ACC-MB-R0:C-USC0805
- added D3, D4: 1N4004, ACC-MB-R0:1N4004
- added D5: 1N4758A - 56Vz, ACC-MB-R0:ZENER-DIODEZD-12.5
- added IC1: 555, ACC-MB-R0:555P
- added OK3: LTV816, ACC-MB-R0:LTV816
- added R10, R13, R4, R6, R8: 1M, ACC-MB-R0:R-US_R0805:1
- added R11: 2.2k, ACC-MB-R0:R-US_R0805:1
- added R12: 4.7M, ACC-MB-R0:R-US_R0805:1
- added R16: 200, ACC-MB-R0:R-US_R2010
- added R17, R19: 10k, ACC-MB-R0:R-US_R0805:1
- added R3, R5, R7, R9: 100, ACC-MB-R0:R-US_R0805:1
- added U$13, U$26: IPBT-102-H1-T-D, ACC-MB-R0:IPBT-102-H1-T-D
- added U$14: PHOENIX_1725724, ACC-MB-R0:PHOENIX_1725724
- added U$15, U$16, U$17, U$18, U$19: BUZ11, ACC-MB-R0:BUZ11
- added U$20, U$21: DCDC_PARTS_282838-2_TE, ACC-MB-R0:DCDC_PARTS_282838-2_TE
- added U$22: _CUSTOM_IXCY10M90SD2PAK, ACC-MB-R0:_CUSTOM_IXCY10M90SD2PAK
- added U$23: MIC4417, ACC-MB-R0:MIC4417
- added U$24, U$25: HSA25, ACC-MB-R0:HSA25
Connections:
- new net ACC_LGHT: U$14.P$7, U$15.D
- new net AIR_ON: D3.C, D4.C, R19.2, R7.1, R8.2, U$15.G, U$23.CTL
- new net DISCHARGE+: U$12.A1, U$12.A10, U$12.A11, U$12.A12, U$12.A13, U$12.A14, U$12.A15, U$12.A16, U$12.A17, U$12.A18, U$12.A2, U$12.A3, U$12.A4, U$12.A5, U$12.A6, U$12.A7, U$12.A8, U$12.A9, U$4.A12, U$4.A13, U$4.A14, U$4.A15, U$4.A16, U$4.A17, U$4.A18
- new net HV+_DRY_FUSED: D5.C, HV+_FUSE_DRY.P$1
- new net N$10: R3.1, R4.2
- new net N$11: R3.2, U$16.G, U$23.GATE
- new net N$12: R5.2, U$17.G
- new net N$13: U$18.S, U$19.D
- new net N$14: D4.A, OK3.EMIT, R17.2
- new net N$15: D3.A, R13.1, U$17.D
- new net N$16: R7.2, U$18.G
- new net N$17: R9.2, U$19.G
- new net N$18: 1A_500V_FUSE_IMD_VSENSE.P$2, U$21.P$2
- new net N$19: 1A_500V_FUSE_ENERGYMETER.P$2, U$21.P$1
- new net N$20: R16.2, U$22.K
- new net N$21: D5.A, U$22.A
- new net N$22: OK3.A, R16.1
- new net N$7: IC1.DIS, R11.1, R12.2
- new net N$8: IC1.OUT, R10.2, R9.1
- new net N$9: C3.1, IC1.TRE, IC1.TRI, R12.1
- new net TSAL_GRN_GND: R5.1, R6.2, U$14.P$5, U$16.D
- new net TSAL_RED_GND: U$14.P$4, U$18.D
- new net V+: HV+_FUSE_DRY.P$2, U$20.P$1, U$26.P$1, U$26.P$2
- new net V-: 1A_500V_FUSE_ENERGYMETER.P$1, 1A_500V_FUSE_IMD_VSENSE.P$1, OK3.C, U$20.P$2, U$22.G, U$26.P$3, U$26.P$4
- net +12V: now also C5.1, C6.1, C7.1, IC1./RES, IC1.VCC+, OK3.COL, R11.2, R13.2, U$14.P$1, U$14.P$3, U$14.P$6, U$23.VS, U$4.A1, U$4.A10, U$4.A11, U$4.A2, U$4.A3, U$4.A4, U$4.A5, U$4.A6, U$4.A7, U$4.A8, U$4.A9
- net GND: now also C3.2, C4.2, C5.2, C6.2, C7.2, IC1.GND, R10.1, R17.1, R19.1, R4.1, R6.1, R8.1, U$12.B1, U$12.B10, U$12.B11, U$12.B12, U$12.B13, U$12.B14, U$12.B15, U$12.B16, U$12.B17, U$12.B18, U$12.B2, U$12.B3, U$12.B4, U$12.B5, U$12.B6, U$12.B7, U$12.B8, U$12.B9, U$14.P$2, U$15.S, U$16.S, U$17.S, U$19.S, U$23.GND
- net N$1: now also C4.1, IC1.CON; no longer D1.C, R1.1
- net N$2: now also C2.2, U$13.P$3, U$13.P$4, U$5.B12, U$5.B13, U$5.B14, U$5.B15, U$5.B16, U$5.B17, U$5.B18; no longer C1.2
- net N$4: now also C1.2, U$4.B12, U$4.B13, U$4.B14, U$4.B15, U$4.B16, U$4.B17, U$4.B18, U$5.B1, U$5.B10, U$5.B11, U$5.B2, U$5.B3, U$5.B4, U$5.B5, U$5.B6, U$5.B7, U$5.B8, U$5.B9
- net N$5: now also D1.C, R1.1, U$13.P$1, U$13.P$2, U$4.B1, U$4.B10, U$4.B11, U$4.B2, U$4.B3, U$4.B4, U$4.B5, U$4.B6, U$4.B7, U$4.B8, U$4.B9; no longer C2.2
Other:
- note added: "+12V POWER"
- note added: "ACC LIGHT"
- note added: "Clock to generate 4hz TSAL signal"
- note added: "Current regulators measure current across each AIR PN: IXCY10M90S"
- note added: "DRY POLE SENSE: HV+ DRY TO HV-DRY"
- note added: "E-METER VSENSE"
- note added: "HIGH VOLTAGE CIRCUIT"
- note added: "IMD VSENSE"
- note added: "IXCY10M90S"
- note added: "If current is detected across AIRs, TSAL is activated."
- note added: "LOW VOLTAGE CIRCUIT"
- note added: "LV Output Terminals"
- note added: "Mosfet to drive green TSAL LED"
- note added: "Mosfets to drive dashboard troubleshooting LEDs, and Accumulator indicator light"
- note added: "Mosfets to drive red TSAL LED"
- note added: "R1 - 100 R2 - 1M R3 - 100 R4 - 1M R5 - 100 R6 - 1M R7 - 100 R8 - 1M R9 - 2.2K R10 - 4.7M R11 - 1M R12 - 200 R13 - 200 ------ C1 - 39n C2 - 10n C3 - 100n"
- note added: "Relays For IMD, AMS"
- note added: "TSAL OUTPUT"
- note added: "TSMP OUTPUT"
- note added: "WARN LIGHTS"
- note added: "X1+"
- note added: "X2-"
- note added: "Zener Diode Vz = 56V: when V > 56V, diode will break down and supply current regulator"

Commit message: update
Parts:
- removed U$13, U$26: IPBT-102-H1-T-D, ACC-MB-R0:IPBT-102-H1-T-D
- removed U$14: PHOENIX_1725724, ACC-MB-R0:PHOENIX_1725724
- removed U$20, U$21: DCDC_PARTS_282838-2_TE, ACC-MB-R0:DCDC_PARTS_282838-2_TE
- added X2, X3, X5: 5566-8, con-molex:5566-8
Connections:
- removed net N$19: 1A_500V_FUSE_ENERGYMETER.P$2, U$21.P$1
- new net N$23: D1.C, R1.1, U$4.B1, U$4.B10, U$4.B11, U$4.B2, U$4.B3, U$4.B4, U$4.B5, U$4.B6, U$4.B7, U$4.B8, U$4.B9, X3-5.S, X3-6.S, X3-7.S, X3-8.S
- net +12V: now also X2-2.S, X2-4.S, X2-8.S; no longer U$14.P$1, U$14.P$3, U$14.P$6
- net ACC_LGHT: now also X2-7.S; no longer U$14.P$7
- net GND: now also X2-1.S, X2-3.S; no longer U$14.P$2
- net N$18: now also X5-7.S; no longer U$21.P$2
- net N$2: now also 1A_500V_FUSE_ENERGYMETER.P$2, X5-3.S; no longer C2.2, U$13.P$3, U$13.P$4, U$5.B12, U$5.B13, U$5.B14, U$5.B15, U$5.B16, U$5.B17, U$5.B18
- net N$5: now also C2.2, U$5.B12, U$5.B13, U$5.B14, U$5.B15, U$5.B16, U$5.B17, U$5.B18, X3-1.S, X3-2.S, X3-3.S, X3-4.S; no longer D1.C, R1.1, U$13.P$1, U$13.P$2, U$4.B1, U$4.B10, U$4.B11, U$4.B2, U$4.B3, U$4.B4, U$4.B5, U$4.B6, U$4.B7, U$4.B8, U$4.B9
- net TSAL_GRN_GND: now also X2-6.S; no longer U$14.P$5
- net TSAL_RED_GND: now also X2-5.S; no longer U$14.P$4
- net V+: now also X5-1.S, X5-5.S; no longer U$20.P$1, U$26.P$1, U$26.P$2
- net V-: now also X5-4.S, X5-8.S; no longer U$20.P$2, U$26.P$3, U$26.P$4
Other:
- note removed: "TSMP OUTPUT"

Commit message: model
Parts:
- removed X2, X3: 5566-8, con-molex:5566-8
- added U$13, U$14: SR4M4012_TE, Main:SR4M4012_TE
- added X1: 5566-24, Main:5566-24
- 1A_500V_FUSE_ENERGYMETER, 1A_500V_FUSE_IMD_VSENSE, HV+_FUSE_DRY: device ACC-MB-R0:_CUSTOM_PARTS_LF_885 -> Main:_CUSTOM_PARTS_LF_885
- C1, C2: device 111_Custom:AIR_HOLDUP_CAP -> Main:AIR_HOLDUP_CAP
- C3, C4, C5, C6, C7: device ACC-MB-R0:C-USC0805 -> Main:C-USC0805
- D1, D2: device 111_Custom:AIR_HOLDUP_DIODE -> Main:AIR_HOLDUP_DIODE
- D3, D4: device ACC-MB-R0:1N4004 -> Main:1N4004
- D5: device ACC-MB-R0:ZENER-DIODEZD-12.5 -> Main:ZENER-DIODEZD-12.5
- H1, H2, H3, H4: device ACC-MB-R0:MOUNT-HOLE5.5 -> Main:MOUNT-HOLE5.5
- IC1: device ACC-MB-R0:555P -> Main:555P
- OK3: device ACC-MB-R0:LTV816 -> Main:LTV816
- R1, R2: device 111_Custom:AIR_HOLDUP_RESISTOR -> Main:AIR_HOLDUP_RESISTOR
- R16: device ACC-MB-R0:R-US_R2010 -> Main:R-US_R2010
- U$1, U$2: device ACC-MB-R0:FUSE_HOLDER -> Main:FUSE_HOLDER
- U$10, U$11, U$12, U$3, U$4, U$5, U$6, U$7, U$8, U$9: device ACC-MB-R0:PCIE-36-CONN -> Main:PCIE-36-CONN
- U$15, U$16, U$17, U$18, U$19: device ACC-MB-R0:BUZ11 -> Main:BUZ11
- U$22: device ACC-MB-R0:_CUSTOM_IXCY10M90SD2PAK -> Main:_CUSTOM_IXCY10M90SD2PAK
- U$23: device ACC-MB-R0:MIC4417 -> Main:MIC4417
- U$24, U$25: device ACC-MB-R0:HSA25 -> Main:HSA25
- X5: device con-molex:5566-8 -> Main:5566-8
Connections:
- removed net N$23: D1.C, R1.1, U$4.B1, U$4.B10, U$4.B11, U$4.B2, U$4.B3, U$4.B4, U$4.B5, U$4.B6, U$4.B7, U$4.B8, U$4.B9, X3-5.S, X3-6.S, X3-7.S, X3-8.S
- new net CH1IN: U$13.NOA2
- new net CH2IN: U$14.NOB2
- new net N$19: U$14.NOB3
- new net PRECHARGE+: U$9.A1, U$9.A10, U$9.A11, U$9.A12, U$9.A13, U$9.A14, U$9.A15, U$9.A16, U$9.A17, U$9.A18, U$9.A2, U$9.A3, U$9.A4, U$9.A5, U$9.A6, U$9.A7, U$9.A8, U$9.A9, X1-14.S
- new net RST1IN: U$13.NOB2, U$14.COIL+
- new net RST2IN: U$13.COIL-, U$14.NOA2
- new net SAFETY+: D1.C, R1.1, U$4.B1, U$4.B10, U$4.B11, U$4.B2, U$4.B3, U$4.B4, U$4.B5, U$4.B6, U$4.B7, U$4.B8, U$4.B9, X1-1.S
- new net SAFETY-: C2.2, U$5.B12, U$5.B13, U$5.B14, U$5.B15, U$5.B16, U$5.B17, U$5.B18, X1-13.S
- net +12V: now also U$13.NOA3; no longer X2-2.S, X2-4.S, X2-8.S
- net ACC_LGHT: now also X1-11.S; no longer X2-7.S
- net GND: now also U$13.COIL+, U$14.COIL-, U$9.B1, U$9.B10, U$9.B11, U$9.B12, U$9.B13, U$9.B14, U$9.B15, U$9.B16, U$9.B17, U$9.B18, U$9.B2, U$9.B3, U$9.B4, U$9.B5, U$9.B6, U$9.B7, U$9.B8, U$9.B9, X1-2.S, X1-24.S; no longer X2-1.S, X2-3.S
- net N$5: now also U$13.NOB3, U$14.NOA3; no longer C2.2, U$5.B12, U$5.B13, U$5.B14, U$5.B15, U$5.B16, U$5.B17, U$5.B18, X3-1.S, X3-2.S, X3-3.S, X3-4.S
- net TSAL_GRN_GND: now also X1-10.S; no longer X2-6.S
- net TSAL_RED_GND: now also X1-12.S; no longer X2-5.S
Other:
- note added: "Monitor Relays"
