File: ACC-MB/Rev1/MainBoard/Main.brd (EAGLE design)
At the start: 210 x 180 mm, 17 parts, among them X11 5566-10, X12 5566-10, X2 5566-10, X3 5566-10, X4 5566-10, X6 5566-10, X7 5566-10, X8 5566-10, X9 5566-4

Commit message: update
Parts:
- removed U$2: FUSE_HOLDER, Main:FUSE_HOLDER
- removed U$5: TO247RESISTORHEATINK, ACC-MB-R0:_CUSTOM_TO-247-2V
- removed X11, X12, X2, X3, X4, X6, X7, X8: 5566-10, con-molex:5566-10
- removed X9: 5566-4, con-molex:5566-4
- added AIR_N_HV, AIR_N_LV, AIR_P_HV, AIR_P_LV, DCDC_HV, DCDC_LV, DIS_PRE_CHARGE_HV, DIS_PRE_CHARGE_LV, HVIB_HV, HVIB_LV: 15-24-7100, ACC-MB-R0:5566-10-BMI
- added INPUT_FUSE: 2.5A, ACC-MB-R0:_CUSTOM_PARTS_LF_885
- added LED1, LED2: (no value), ACC-MB-R0:LED3MM
- added R1, R4: (no value), ACC-MB-R0:R0805
- added U$4: (no value), ACC-MB-R0:_CUSTOM_TO-247-2V
- added X13: 5566-4, ACC-MB-R0:5566-4
- U$1: value FUSE_HOLDER -> MAINFUSEASSY; device Main:FUSE_HOLDER -> ACC-MB-R0:MAINFUSEASSY
- U$3: value TO247RESISTORHEATINK -> (none)
- moved U$1 94.0 mm to (10.0, 61.0)
- moved U$3 28.8 mm to (172.0, 131.0)
Connections:
- removed net N$25: X6.10, X6.5
- removed net N$26: X6.4, X6.9
- removed net N$29: X6.1, X6.3, X6.6, X6.8
- removed net N$4: X2.4, X2.9
- removed net N$6: X2.3, X2.8
- new net ACC_LGHT: HVIB_LV.1
- new net DISCHARGE: DIS_PRE_CHARGE_LV.1, DIS_PRE_CHARGE_LV.2
- new net HV-_DRY_AUX: DIS_PRE_CHARGE_HV.10, DIS_PRE_CHARGE_HV.5, X13.4
- new net N$1: HVIB_LV.6
- new net N$12: HVIB_LV.4
- new net N$16: HVIB_LV.5
- new net N$2: LED2.K, R1.2
- new net N$5: LED1.K, R4.2
- new net PRECHARGE_SIG: DIS_PRE_CHARGE_LV.6, DIS_PRE_CHARGE_LV.7
- new net TSAL_GRN_GND: HVIB_LV.2
- new net TSAL_RED_GND: HVIB_LV.3
- net +12V: now also DCDC_LV.10, DCDC_LV.6, DCDC_LV.7, DCDC_LV.9, DIS_PRE_CHARGE_LV.10, DIS_PRE_CHARGE_LV.9, HVIB_LV.10, HVIB_LV.8, HVIB_LV.9, LED1.A, LED2.A; no longer X11.10, X11.4, X11.5, X11.9
- net DCDC_EN: now also DCDC_LV.8; no longer X11.8
- net GND: now also AIR_N_LV.1, AIR_N_LV.3, AIR_N_LV.6, AIR_N_LV.8, AIR_P_LV.3, AIR_P_LV.8, DCDC_LV.1, DCDC_LV.2, DCDC_LV.3, DCDC_LV.4, DCDC_LV.5, DIS_PRE_CHARGE_LV.3, DIS_PRE_CHARGE_LV.4, DIS_PRE_CHARGE_LV.5, HVIB_LV.7, R1.1, R4.1; no longer X11.1, X11.2, X11.6, X11.7
- net HV+_DRY: now also AIR_P_HV.1, AIR_P_HV.2, AIR_P_HV.6, AIR_P_HV.7, DCDC_HV.1, DCDC_HV.6, DIS_PRE_CHARGE_HV.1, DIS_PRE_CHARGE_HV.6, HVIB_HV.1, HVIB_HV.6, INPUT_FUSE.P$1, U$3.1; no longer U$5.2, X12.1, X12.2, X12.6, X12.7, X3.10, X3.4, X3.5, X3.9, X7.1, X7.6
- net HV+_WET: now also AIR_P_HV.10, AIR_P_HV.4, AIR_P_HV.5, AIR_P_HV.9, DIS_PRE_CHARGE_HV.3, DIS_PRE_CHARGE_HV.8; no longer X3.1, X3.2, X3.6, X3.7, X7.3, X7.8
- net HV-_DRY: now also AIR_N_HV.10, AIR_N_HV.4, AIR_N_HV.5, AIR_N_HV.9, DCDC_HV.10, DCDC_HV.5, HVIB_HV.10, HVIB_HV.5, U$4.1; no longer U$3.2, X12.10, X12.4, X12.5, X12.9, X4.10, X4.4, X4.5, X4.9, X7.10, X7.5
- net HV-_WET: now also AIR_N_HV.1, AIR_N_HV.2, AIR_N_HV.6, AIR_N_HV.7; no longer X4.1, X4.2, X4.6, X4.7
- net N$23: now also U$3.2, X13.1; no longer U$5.1, X9.1
- net N$24: now also U$4.2, X13.2; no longer U$3.1, X9.4
- net N$3: now also INPUT_FUSE.P$2, X13.3; no longer X2.10, X2.5
- net SAFETY+: now also AIR_P_LV.4, AIR_P_LV.9; no longer X2.2, X2.7
- net SAFETY-: now also AIR_N_LV.2, AIR_N_LV.7, AIR_P_LV.10, AIR_P_LV.5; no longer X2.1, X2.6, X6.2, X6.7
Routing:
- net HV+_DRY: track 0.00 -> 249.7 mm
- net HV-_DRY: track 0.00 -> 222.5 mm
- net HV+_WET: track 0.00 -> 119.4 mm
- net HV-_DRY_AUX: track 0.00 -> 91.8 mm
- net N$23: track 0.00 -> 29.5 mm
- net N$24: track 0.00 -> 25.5 mm
- net N$3: track 0.00 -> 18.9 mm
- net N$5: track 0.00 -> 6.92 mm
- net N$2: track 0.00 -> 6.92 mm
- added copper zone on layer 1, net +12V
- added copper zone on layer 16, net GND
Other:
- board text removed: "AIR+"
- board text removed: "Discharge"

Commit message: update
Parts:
- added X1: 5566-24, ACC-MB-R0:5566-24
- moved LED1 63.0 mm to (29.0, 10.0)
- moved R4 63.0 mm to (29.0, 4.00)
- moved DIS_PRE_CHARGE_HV 16.0 mm to (120.0, 165.0)
- moved DIS_PRE_CHARGE_LV 16.0 mm to (120.0, 15.0)
- moved AIR_N_HV 3.00 mm to (40.0, 100.0)
- moved AIR_N_LV 3.00 mm to (40.0, 15.0)
Connections:
- net ACC_LGHT: now also X1.24
- net TSAL_GRN_GND: now also X1.23
- net TSAL_RED_GND: now also X1.22
Routing:
- net HV+_DRY: track 249.7 -> 232.0 mm
- net HV+_WET: track 119.4 -> 135.4 mm
- net HV-_DRY_AUX: track 91.8 -> 107.8 mm
- net HV-_DRY: track 222.5 -> 223.8 mm
