File: ACC-MB/Rev1/MainBoard/Main.sch (EAGLE design)
At the start: 17 parts, among them X11 5566-10, X12 5566-10, X2 5566-10, X3 5566-10, X4 5566-10, X6 5566-10, X7 5566-10, X8 5566-10, X9 5566-4

Commit message: update
Parts:
- removed U$2: FUSE_HOLDER, Main:FUSE_HOLDER
- removed U$5: TO247RESISTORHEATINK, ACC-MB-R0:TO247RESISTORHEATINK
- removed X11, X12, X2, X3, X4, X6, X7, X8: 5566-10, con-molex:5566-10
- removed X9: 5566-4, con-molex:5566-4
- added AIR_N_HV, AIR_N_LV, AIR_P_HV, AIR_P_LV, DCDC_HV, DCDC_LV, DIS_PRE_CHARGE_HV, DIS_PRE_CHARGE_LV, HVIB_HV, HVIB_LV: 15-24-7100, ACC-MB-R0:15-24-7100
- added INPUT_FUSE: 2.5A, ACC-MB-R0:_CUSTOM_PARTS_LF_885
- added LED1, LED2: (no value), ACC-MB-R0:LED3MM
- added R1, R4: (no value), ACC-MB-R0:R-US_R0805
- added U$4: TO247RESISTORHEATINK, ACC-MB-R0:TO247RESISTORHEATINK
- added X13: 5566-4, ACC-MB-R0:5566-4
- U$1: value FUSE_HOLDER -> MAINFUSEASSY; device Main:FUSE_HOLDER -> ACC-MB-R0:MAINFUSEASSY
Connections:
- removed net N$25: X6-10.S, X6-5.S
- removed net N$26: X6-4.S, X6-9.S
- removed net N$29: X6-1.S, X6-3.S, X6-6.S, X6-8.S
- removed net N$4: X2-4.S, X2-9.S
- removed net N$6: X2-3.S, X2-8.S
- new net ACC_LGHT: HVIB_LV.1
- new net DISCHARGE: DIS_PRE_CHARGE_LV.1, DIS_PRE_CHARGE_LV.2
- new net HV-_DRY_AUX: DIS_PRE_CHARGE_HV.10, DIS_PRE_CHARGE_HV.5, X13-4.S
- new net N$1: HVIB_LV.6
- new net N$12: HVIB_LV.4
- new net N$16: HVIB_LV.5
- new net N$2: LED2.C, R1.2
- new net N$5: LED1.C, R4.2
- new net PRECHARGE_SIG: DIS_PRE_CHARGE_LV.6, DIS_PRE_CHARGE_LV.7
- new net TSAL_GRN_GND: HVIB_LV.2
- new net TSAL_RED_GND: HVIB_LV.3
- net +12V: now also DCDC_LV.10, DCDC_LV.6, DCDC_LV.7, DCDC_LV.9, DIS_PRE_CHARGE_LV.10, DIS_PRE_CHARGE_LV.9, HVIB_LV.10, HVIB_LV.8, HVIB_LV.9, LED1.A, LED2.A; no longer X11-10.S, X11-4.S, X11-5.S, X11-9.S
- net DCDC_EN: now also DCDC_LV.8; no longer X11-8.S
- net GND: now also AIR_N_LV.1, AIR_N_LV.3, AIR_N_LV.6, AIR_N_LV.8, AIR_P_LV.3, AIR_P_LV.8, DCDC_LV.1, DCDC_LV.2, DCDC_LV.3, DCDC_LV.4, DCDC_LV.5, DIS_PRE_CHARGE_LV.3, DIS_PRE_CHARGE_LV.4, DIS_PRE_CHARGE_LV.5, HVIB_LV.7, R1.1, R4.1; no longer X11-1.S, X11-2.S, X11-6.S, X11-7.S
- net HV+_DRY: now also AIR_P_HV.1, AIR_P_HV.2, AIR_P_HV.6, AIR_P_HV.7, DCDC_HV.1, DCDC_HV.6, DIS_PRE_CHARGE_HV.1, DIS_PRE_CHARGE_HV.6, HVIB_HV.1, HVIB_HV.6, INPUT_FUSE.P$1, U$3.P$1; no longer U$5.P$2, X12-1.S, X12-2.S, X12-6.S, X12-7.S, X3-10.S, X3-4.S, X3-5.S, X3-9.S, X7-1.S, X7-6.S
- net HV+_WET: now also AIR_P_HV.10, AIR_P_HV.4, AIR_P_HV.5, AIR_P_HV.9, DIS_PRE_CHARGE_HV.3, DIS_PRE_CHARGE_HV.8; no longer X3-1.S, X3-2.S, X3-6.S, X3-7.S, X7-3.S, X7-8.S
- net HV-_DRY: now also AIR_N_HV.10, AIR_N_HV.4, AIR_N_HV.5, AIR_N_HV.9, DCDC_HV.10, DCDC_HV.5, HVIB_HV.10, HVIB_HV.5, U$4.P$1; no longer U$3.P$2, X12-10.S, X12-4.S, X12-5.S, X12-9.S, X4-10.S, X4-4.S, X4-5.S, X4-9.S, X7-10.S, X7-5.S
- net HV-_WET: now also AIR_N_HV.1, AIR_N_HV.2, AIR_N_HV.6, AIR_N_HV.7; no longer X4-1.S, X4-2.S, X4-6.S, X4-7.S
- net N$23: now also U$3.P$2, X13-1.S; no longer U$5.P$1, X9-1.S
- net N$24: now also U$4.P$2, X13-2.S; no longer U$3.P$1, X9-4.S
- net N$3: now also INPUT_FUSE.P$2, X13-3.S; no longer X2-10.S, X2-5.S
- net SAFETY+: now also AIR_P_LV.4, AIR_P_LV.9; no longer X2-2.S, X2-7.S
- net SAFETY-: now also AIR_N_LV.2, AIR_N_LV.7, AIR_P_LV.10, AIR_P_LV.5; no longer X2-1.S, X2-6.S, X6-2.S, X6-7.S
Other:
- note added: "HVIB"

Commit message: update
Parts:
- added X1: 5566-24, ACC-MB-R0:5566-24
Connections:
- net ACC_LGHT: now also X1-24.S
- net TSAL_GRN_GND: now also X1-23.S
- net TSAL_RED_GND: now also X1-22.S
Changed lines of the file:
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@@
 <part name="GND9" library="ACC-MB-R0" library_urn="urn:adsk.eagle:library:13208985" deviceset="GND" device=""/>
 <part name="INPUT_FUSE" library="ACC-MB-R0" deviceset="_CUSTOM_PARTS_LF_885" device="" package3d_urn="urn:adsk.eagle:package:13209479/2" value="2.5A"/>
+<part name="X1" library="ACC-MB-R0" library_urn="urn:adsk.eagle:library:13208985" deviceset="5566-24" device="" package3d_urn="urn:adsk.eagle:package:14396841/2"/>
 </parts>
 <sheets>
@@
 <instance part="GND9" gate="1" x="63.5" y="191.77"/>
 <instance part="INPUT_FUSE" gate="G$1" x="134.62" y="180.34"/>
+<instance part="X1" gate="-1" x="254" y="109.22"/>
+<instance part="X1" gate="-2" x="254" y="106.68"/>
+<instance part="X1" gate="-3" x="254" y="104.14"/>
+<instance part="X1" gate="-4" x="254" y="101.6"/>
+<instance part="X1" gate="-5" x="254" y="99.06"/>
+<instance part="X1" gate="-6" x="254" y="96.52"/>
+<instance part="X1" gate="-7" x="254" y="93.98"/>
+<instance part="X1" gate="-8" x="254" y="91.44"/>
+<instance part="X1" gate="-9" x="254" y="88.9"/>
+<instance part="X1" gate="-10" x="254" y="86.36"/>
+<instance part="X1" gate="-11" x="254" y="83.82"/>
+<instance part="X1" gate="-12" x="254" y="81.28"/>
+<instance part="X1" gate="-13" x="254" y="78.74"/>
+<instance part="X1" gate="-14" x="254" y="76.2"/>
+<instance part="X1" gate="-15" x="254" y="73.66"/>
+<instance part="X1" gate="-16" x="254" y="71.12"/>
+<instance part="X1" gate="-17" x="254" y="68.58"/>
+<instance part="X1" gate="-18" x="254" y="66.04"/>
+<instance part="X1" gate="-19" x="254" y="63.5"/>
+<instance part="X1" gate="-20" x="254" y="60.96"/>
+<instance part="X1" gate="-21" x="254" y="58.42"/>
+<instance part="X1" gate="-22" x="254" y="55.88"/>
+<instance part="X1" gate="-23" x="254" y="53.34"/>
+<instance part="X1" gate="-24" x="254" y="50.8"/>
 </instances>
 <busses>
@@
 <junction x="330.2" y="48.26"/>
 </segment>
+<segment>
+<label x="226.06" y="53.34" size="1.778" layer="95"/>
+<wire x1="251.46" y1="53.34" x2="224.79" y2="53.34" width="0.1524" layer="91"/>
+<pinref part="X1" gate="-23" pin="S"/>
+</segment>
 </net>
 <net name="TSAL_RED_GND" class="0">
@@
 <wire x1="330.2" y1="50.8" x2="303.53" y2="50.8" width="0.1524" layer="91"/>
 <junction x="330.2" y="50.8"/>
+</segment>
+<segment>
+<label x="226.06" y="55.88" size="1.778" layer="95"/>
+<wire x1="251.46" y1="55.88" x2="224.79" y2="55.88" width="0.1524" layer="91"/>
+<pinref part="X1" gate="-22" pin="S"/>
 </segment>
 </net>
@@
 <junction x="330.2" y="45.72"/>
 </segment>
-</net>
+<segment>
+<label x="226.06" y="50.8" size="1.778" layer="95"/>
+<wire x1="251.46" y1="50.8" x2="226.06" y2="50.8" width="0.1524" layer="91"/>
+<pinref part="X1" gate="-24" pin="S"/>
+</segment>
+</net>
