File: ACC-MB/Rev3/HVIBDC/HVIBDC.brd (EAGLE design)
At the start: 92 x 64 mm, 49 parts, among them IC1 555

Commit message: d
Routing:
- net AIR_ON: track 69.6 -> 80.8 mm
- net N$22: track 9.24 -> 8.24 mm
Other:
- outline, holes or cut-outs redrawn
- board text added: "+12V"
- board text added: "<1A"
- board text added: "ACC"
- board text added: "GND"
- board text added: "GRN"
- board text added: "HV+ HV-"
- board text added: "RED"
- board text added: "REV3, BUILD1"
- board text added: "Vz = 60V"
- board text added: "WESTERN FORMULA RACING"
- board text removed: "1"
- board text removed: "1 - + 12V 2 - GND 3 - +12V TSAL 4 - GND RD 5 - GND GR 6 - +12V ACC 7 - GND ACC"

Commit message: stuff
Parts:
- removed PRECHAGE, PRECHAGE1, PRECHAGE2, PRECHAGE3: (no value), ACC-MB-R0:LED3MM
- removed U$5: 3568FUSEHOLDER, ACC-MB-R0:3568
- added ACC, GREEN, PWR, RED: (no value), ACC-MB-R0:CHIPLED_0805
- moved LEDR4 20.2 mm to (11.0, 37.0)
- moved D5 2.68 mm to (80.6, 54.2)
- moved U$22 2.40 mm to (72.7, 57.2)
- moved D3 1.70 mm to (90.2, 54.2)
- moved D6 1.70 mm to (83.8, 54.2)
- moved D2 1.20 mm to (87.0, 54.2)
- moved R16 1.08 mm to (75.0, 47.6)
- moved LEDR2 1.00 mm to (14.0, 37.0)
Connections:
- removed net N$11: U$2.10, U$2.8, U$2.9, U$5.L1, U$5.L2
- net +12V: now also ACC.A, GREEN.A, PWR.A, RED.A, U$2.10, U$2.8, U$2.9; no longer PRECHAGE.A, PRECHAGE1.A, PRECHAGE2.A, PRECHAGE3.A, U$5.R1, U$5.R2
- net N$10: now also ACC.C; no longer PRECHAGE.K
- net N$12: now also GREEN.C; no longer PRECHAGE1.K
- net N$16: now also RED.C; no longer PRECHAGE2.K
- net N$17: now also PWR.C; no longer PRECHAGE3.K
Routing:
- net N$11: track 58.7 -> 0.00 mm
- net N$16: track 2.78 -> 28.5 mm
- net +12V: track 86.1 -> 111.2 mm
- net N$17: track 2.78 -> 27.9 mm
- net N$12: track 2.78 -> 27.6 mm, vias 0 -> 1
- net N$10: track 2.78 -> 27.6 mm, vias 0 -> 1
- net N$20: track 4.38 -> 2.75 mm
- net V-: track 59.7 -> 59.1 mm
Other:
- board text added: "HV+"
- board text added: "HV-"
- board text added: "NC"

Commit message: g
Routing:
- net +12V: track 111.2 -> 117.4 mm, vias 2 -> 4
Changed lines of the file:
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@@
 <wire x1="30" y1="61" x2="31" y2="60" width="0.2" layer="1"/>
 <wire x1="31" y1="60" x2="31" y2="47.4" width="0.2" layer="1"/>
-<wire x1="12" y1="18.29" x2="7.8" y2="18.29" width="0" layer="19" extent="1-1"/>
+<wire x1="12" y1="18.29" x2="12" y2="16.2" width="0.6096" layer="16"/>
+<via x="11.4" y="15.6" extent="1-16" drill="0.35"/>
+<wire x1="11.4" y1="15.6" x2="8.1" y2="15.6" width="0.6096" layer="1"/>
+<via x="8.1" y="15.6" extent="1-16" drill="0.35"/>
+<wire x1="12" y1="16.2" x2="11.4" y2="15.6" width="0.6096" layer="16"/>
 </signal>
 <signal name="AIR_ON">
@@
 <contactref element="U$10" pad="2"/>
 <contactref element="U$2" pad="1"/>
-<wire x1="59" y1="22.35" x2="58.0856" y2="21.4356" width="1.27" layer="16"/>
-<wire x1="58.0856" y1="21.4356" x2="58.0856" y2="20.83845" width="1.27" layer="16"/>
-<wire x1="58.0856" y1="20.83845" x2="55.24715" y2="18" width="1.27" layer="16"/>
-<wire x1="55.24715" y1="18" x2="28.15" y2="18" width="1.27" layer="16"/>
+<wire x1="59" y1="22.35" x2="58.9856" y2="22.3356" width="1.27" layer="16"/>
+<wire x1="58.9856" y1="22.3356" x2="58.9856" y2="21.13845" width="1.27" layer="16"/>
+<wire x1="58.9856" y1="21.13845" x2="55.84715" y2="18" width="1.27" layer="16"/>
+<wire x1="55.84715" y1="18" x2="28.15" y2="18" width="1.27" layer="16"/>
 <wire x1="28.15" y1="18" x2="22.94" y2="12.79" width="1.27" layer="16"/>
 <wire x1="22.94" y1="12.79" x2="20.4" y2="12.79" width="1.27" layer="16"/>

Commit message: update
Changed lines of the file:
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@@
 <text x="69.6" y="26.5" size="1" layer="21">HIGH VOLTAGE</text>
 <wire x1="0" y1="61" x2="0" y2="3" width="0" layer="20"/>
-<wire x1="67.09" y1="-2.497" x2="67.09" y2="67.345" width="4" layer="21"/>
-<wire x1="67.09" y1="67.345" x2="67.193" y2="67.448" width="4" layer="21"/>
 <text x="64" y="49" size="2.54" layer="26" rot="MR0">WESTERN FORMULA RACING</text>
 <text x="40" y="61" size="1.778" layer="26" rot="MR0">REV3, BUILD1</text>
@@
 <text x="73" y="22" size="1.778" layer="25">HV-</text>
 <text x="79" y="21" size="1.778" layer="25">NC</text>
+<wire x1="67.2" y1="63.6" x2="67.2" y2="1.2" width="4" layer="25"/>
+<wire x1="67.2" y1="1.2" x2="67.2" y2="63.6" width="4" layer="26"/>
 </plain>
 <attributes>
