File: ACC-MB/Rev3/MainBoard/Main.sch (EAGLE design)
At the start: 80 parts, among them T1 2N2222, X1 5566-24, X2 5566-4, X3 5566-4

Commit message: d
Connections:
- new net INT_FAULT_LED: U$2.NCB4, X1-9.S
- net +12V: no longer DIS_PRE_CHARGE_LV.7
- net N$4: now also U$2.NCA4
- net V+: now also DIS_PRE_CHARGE_HV.4, DIS_PRE_CHARGE_HV.9
- net V-: now also DIS_PRE_CHARGE_HV.2, DIS_PRE_CHARGE_HV.7
Changed lines of the file:
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@@
 </class>
 <class number="2" name="HV" width="1.27" drill="0">
-<clearance class="0" value="1.5"/>
-<clearance class="1" value="1.5"/>
-<clearance class="2" value="1.5"/>
+<clearance class="0" value="1.6"/>
+<clearance class="1" value="1.6"/>
+<clearance class="2" value="1.6"/>
 </class>
 </classes>
@@
 </segment>
 <segment>
-<pinref part="DIS_PRE_CHARGE_LV" gate="G$1" pin="7"/>
-<wire x1="121.92" y1="86.36" x2="119.38" y2="86.36" width="0.1524" layer="91"/>
 <wire x1="119.38" y1="86.36" x2="116.84" y2="86.36" width="0.1524" layer="91"/>
 <wire x1="116.84" y1="86.36" x2="114.3" y2="86.36" width="0.1524" layer="91"/>
 <pinref part="DIS_PRE_CHARGE_LV" gate="G$1" pin="8"/>
-<junction x="119.38" y="86.36"/>
 <pinref part="DIS_PRE_CHARGE_LV" gate="G$1" pin="9"/>
 <junction x="116.84" y="86.36"/>
@@
 <junction x="109.22" y="121.92"/>
 <pinref part="P+7" gate="1" pin="V+"/>
+<pinref part="DIS_PRE_CHARGE_HV" gate="G$1" pin="9"/>
+<wire x1="111.76" y1="121.92" x2="114.3" y2="121.92" width="0.1524" layer="91"/>
+<junction x="111.76" y="121.92"/>
+<pinref part="DIS_PRE_CHARGE_HV" gate="G$1" pin="4"/>
+<wire x1="114.3" y1="109.22" x2="111.76" y2="109.22" width="0.1524" layer="91"/>
+<junction x="111.76" y="109.22"/>
 </segment>
 <segment>
@@
 <wire x1="124.46" y1="109.22" x2="124.46" y2="124.46" width="0.1524" layer="91"/>
 <junction x="124.46" y="124.46"/>
+<pinref part="DIS_PRE_CHARGE_HV" gate="G$1" pin="2"/>
+<wire x1="119.38" y1="109.22" x2="121.92" y2="109.22" width="0.1524" layer="91"/>
+<junction x="121.92" y="109.22"/>
+<pinref part="DIS_PRE_CHARGE_HV" gate="G$1" pin="7"/>
+<wire x1="119.38" y1="121.92" x2="121.92" y2="121.92" width="0.1524" layer="91"/>
+<junction x="121.92" y="121.92"/>
 </segment>
 <segment>
@@
 </segment>
 </net>
+<net name="INT_FAULT_LED" class="0">
+<segment>
+<pinref part="X1" gate="-9" pin="S"/>
+<wire x1="106.68" y1="200.66" x2="81.28" y2="200.66" width="0.1524" layer="91"/>
+<label x="81.28" y="200.66" size="1.778" layer="95"/>
+</segment>
+</net>
 </nets>
 </sheet>
@@
 <wire x1="-85.09" y1="104.14" x2="-81.28" y2="104.14" width="0.1524" layer="91"/>
 <junction x="-85.09" y="105.41"/>
+<pinref part="U$2" gate="G$1" pin="NCA4"/>
+<wire x1="-85.09" y1="105.41" x2="-85.09" y2="106.68" width="0.1524" layer="91"/>
+<wire x1="-85.09" y1="106.68" x2="-81.28" y2="106.68" width="0.1524" layer="91"/>
 </segment>
 </net>
@@
 </segment>
 </net>
+<net name="INT_FAULT_LED" class="0">
+<segment>
+<pinref part="U$2" gate="G$1" pin="NCB4"/>
+<wire x1="-66.04" y1="106.68" x2="-60.96" y2="106.68" width="0.1524" layer="91"/>
+<wire x1="-60.96" y1="106.68" x2="-60.96" y2="134.62" width="0.1524" layer="91"/>
+<wire x1="-60.96" y1="134.62" x2="-38.1" y2="134.62" width="0.1524" layer="91"/>
+<label x="-48.26" y="134.62" size="1.778" layer="95"/>
+</segment>
+</net>

Commit message: stuff
Parts:
- added +12V_SAFE1: (no value), ACC-MB-R0:LEDCHIP-LED0805
- added D1, D2, D3, D4: 1N4007RLG, ACC-MB-R0:1N4004
- added INPUT_FUSE3: 088502.5DR, ACC-MB-R0:_CUSTOM_PARTS_LF_885
- added R1, R2, R5, R6: (no value), ACC-MB-R0:R-US_R0805
- added R3: 10K, ACC-MB-R0:R-US_M0805
- added R4: 2.2K, ACC-MB-R0:R-US_M0805
- added R7: 200, Main:R-US_R2010
- added T2: 2N2222, adafruit:2N2222
- added U$14: 3568FUSEHOLDER, ACC-MB-R0:3568FUSEHOLDER
- added U$22: _CUSTOM_IXCY10M90SD2PAK, Main:_CUSTOM_IXCY10M90SD2PAK
- +12V, +12V_, +12V_SAFE, AMS_OK, EXT1, EXT2, EXT_IN, PRECHARGE_EN, PRECHARGE_OK: device ACC-MB-R0:LED3MM -> ACC-MB-R0:LEDCHIP-LED0805
Connections:
- new net AMS_OK_GND: T2.C, U$13.12
- new net HV-_ORED: +12V_SAFE1.C, D2.A, D3.A, HVIB_HV.10, HVIB_HV.4, HVIB_HV.5, HVIB_HV.9, INPUT_FUSE3.P$2, U$22.G
- new net N$25: DIS_PRE_CHARGE_LV.6, R1.2, R2.2
- new net N$27: R3.2, T2.B
- new net N$29: R5.2, U$12.1
- new net N$30: R6.2, U$13.1
- new net N$31: R7.2, U$22.K
- new net N$41: +12V_SAFE1.A, R7.1
- new net N$42: HVIB_LV.10, HVIB_LV.8, HVIB_LV.9, U$14.1A, U$14.1B
- new net N$44: D1.A, D4.A, INPUT_FUSE3.P$1
- net +12V: now also R5.1, R6.1, U$14.2A, U$14.2B; no longer HVIB_LV.10, HVIB_LV.8, HVIB_LV.9, U$12.1
- net AMS_OK: now also R3.1, R4.2; no longer U$13.12
- net GND: now also R4.1, T2.E; no longer U$13.1
- net HV-_DRY_AUX: now also D1.C, D4.C
- net PRECHARGE_EN: now also R1.1; no longer DIS_PRE_CHARGE_LV.6
- net PRECHARGE_OK: now also R2.1
- net V+: now also U$22.A
- net V-: now also D2.C, D3.C; no longer HVIB_HV.10, HVIB_HV.4, HVIB_HV.5, HVIB_HV.9
Other:
- note added: "IXCY10M90S"
- moved on the sheet: AMS_OK, DIS_PRE_CHARGE_LV, LED_R6

Commit message: g
Parts:
- +12V_SAFE1: device ACC-MB-R0:LEDCHIP-LED0805 -> ACC-MB-R0:LED5MM
Changed lines of the file:
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@@
 <part name="R7" library="Main" library_urn="urn:adsk.eagle:library:14107900" deviceset="R-US_" device="R2010" package3d_urn="urn:adsk.eagle:package:14108443/1" value="200"/>
 <part name="P+18" library="ACC-MB-R0" library_urn="urn:adsk.eagle:library:13324935" deviceset="V+" device=""/>
-<part name="+12V_SAFE1" library="ACC-MB-R0" library_urn="urn:adsk.eagle:library:13208985" deviceset="LED" device="CHIP-LED0805" package3d_urn="urn:adsk.eagle:package:15818/2"/>
+<part name="+12V_SAFE1" library="ACC-MB-R0" library_urn="urn:adsk.eagle:library:13208985" deviceset="LED" device="5MM" package3d_urn="urn:adsk.eagle:package:15799/2"/>
 </parts>
 <sheets>
