File: ACC-MB/Rev3/MainBoard/Main.brd (EAGLE design)
At the start: 210 x 180 mm, 81 parts, among them T1 2N2222, X1 5566-24, X2 5566-4, X3 5566-4

Commit message: d
Parts:
- moved X3 4.03 mm to (143.5, 154.0)
Connections:
- new net INT_FAULT_LED: U$2.NCB4, X1.9
- net +12V: no longer DIS_PRE_CHARGE_LV.7
- net N$4: now also U$2.NCA4
- net V+: now also DIS_PRE_CHARGE_HV.4, DIS_PRE_CHARGE_HV.9
- net V-: now also DIS_PRE_CHARGE_HV.2, DIS_PRE_CHARGE_HV.7
Routing:
- net INT_FAULT_LED: track 0.00 -> 58.0 mm
- net N$4: track 63.0 -> 80.9 mm
- net INT_RST1: track 122.5 -> 127.7 mm
- net +12V_SAFE: track 208.5 -> 211.0 mm
- net N$26: track 84.6 -> 82.4 mm
- added copper zone on layer 1, net V+
- added copper zone on layer 1, net V-
Other:
- outline, holes or cut-outs redrawn
- board text added: "ACCUMULATOR MOTHERBOARD REV3, BUILD1. CONTACT: ANDREW RANDELL"
- board text added: "AIR+, PRECHARGE"
- board text added: "AIR-, DISCHARGE"
- board text added: "DCDC"
- board text added: "EM+"
- board text added: "HIGH VOLTAGE 60~600V"
- board text added: "HV-_AUX"
- board text added: "HVIB"
- board text added: "IMD 12V"
- board text added: "IMD 12V FUSE"
- board text added: "IMD HS"
- board text added: "IMD HV"
- board text added: "IMD LS"
- board text added: "IMD LV"
- board text added: "IMD STATUS"
- board text added: "LOW VOLTAGE <60V"
- board text added: "LV CONN 24"
- board text added: "SAF 12V FUSE"
- board text added: "TSMP+"
- board text added: "TSMP-"
- board text added: "WESTERN FORMULA RACING"
- board text added: "WFR-FSAE 2019-2020"
- board text added: "bottom row: 13: ACC LIGHT 14: TSAL GREEN 15: TSAL RED 16: IMD DATA 17: IMD DATA 18: NC 19,20:AMS +12V ...: GND"
- board text added: "top row: 1: +12V SAFE 2: PRECHARGE EN 3: PRECHARGE OK 4: SAF MAIN OUT 5: EXT RST1 6: EXT RST2 7: AMS OK 8: SAF EXT IN 9: EXT FAULT LED 10, 11, 12: +12V"

Commit message: stuff
Parts:
- added +12V_SAFE1: (no value), ACC-MB-R0:CHIP-LED0805
- added D1, D2, D3, D4: 1N4007RLG, ACC-MB-R0:DO41-10
- added INPUT_FUSE3: 088502.5DR, ACC-MB-R0:_CUSTOM_PARTS_LF_885
- added R1, R2, R5, R6: (no value), ACC-MB-R0:R0805
- added R3: 10K, ACC-MB-R0:M0805
- added R4: 2.2K, ACC-MB-R0:M0805
- added R7: 200, Main:R2010
- added T2: 2N2222, adafruit:TO92-EBC-OVAL
- added U$14: 3568FUSEHOLDER, ACC-MB-R0:3568
- added U$22: _CUSTOM_IXCY10M90SD2PAK, Main:TO228P991X238-3
- +12V, +12V_, +12V_SAFE, AMS_OK, EXT1, EXT2, EXT_IN, PRECHARGE_EN, PRECHARGE_OK: device ACC-MB-R0:LED3MM -> ACC-MB-R0:CHIP-LED0805
- moved R17 29.4 mm to (175.0, 162.0), turned to 270 degrees
- moved R18 22.0 mm to (171.0, 155.0)
- moved +12V 17.3 mm to (165.8, 104.0)
- moved LED_R1 17.3 mm to (170.2, 102.2)
- moved LED_R6 13.1 mm to (84.0, 20.5)
- moved R19 11.4 mm to (167.5, 148.0), turned to 270 degrees
- moved AMS_OK 10.2 mm to (82.0, 19.0)
- moved HVIB_HV 10.0 mm to (157.0, 165.0)
- moved HVIB_LV 10.0 mm to (157.0, 96.0)
- moved X3 7.38 mm to (137.0, 157.5)
- moved LED_R5 6.18 mm to (187.5, 11.5), flipped to the top, turned to 270 degrees
- moved EXT2 1.12 mm to (91.0, 24.0), turned to 180 degrees
- moved EXT1 0.50 mm to (100.5, 25.2), turned to 180 degrees
- moved LED_R3 0.50 mm to (172.2, 13.0)
Connections:
- new net AMS_OK_GND: T2.C, U$13.12
- new net HV-_ORED: +12V_SAFE1.C, D2.A, D3.A, HVIB_HV.10, HVIB_HV.4, HVIB_HV.5, HVIB_HV.9, INPUT_FUSE3.P$2, U$22.1
- new net N$25: DIS_PRE_CHARGE_LV.6, R1.2, R2.2
- new net N$27: R3.2, T2.B
- new net N$29: R5.2, U$12.1
- new net N$30: R6.2, U$13.1
- new net N$31: R7.2, U$22.2
- new net N$41: +12V_SAFE1.A, R7.1
- new net N$42: HVIB_LV.10, HVIB_LV.8, HVIB_LV.9, U$14.L1, U$14.L2
- new net N$44: D1.A, D4.A, INPUT_FUSE3.P$1
- net +12V: now also R5.1, R6.1, U$14.R1, U$14.R2; no longer HVIB_LV.10, HVIB_LV.8, HVIB_LV.9, U$12.1
- net AMS_OK: now also R3.1, R4.2; no longer U$13.12
- net GND: now also R4.1, T2.E; no longer U$13.1
- net HV-_DRY_AUX: now also D1.C, D4.C
- net N$11: now also AMS_OK.C; no longer AMS_OK.K
- net N$13: now also EXT1.C; no longer EXT1.K
- net N$14: now also EXT2.C; no longer EXT2.K
- net N$15: now also EXT_IN.C; no longer EXT_IN.K
- net N$2: now also +12V.C; no longer +12V.K
- net N$5: now also +12V_.C; no longer +12V_.K
- net N$6: now also +12V_SAFE.C; no longer +12V_SAFE.K
- net N$7: now also PRECHARGE_EN.C; no longer PRECHARGE_EN.K
- net N$8: now also PRECHARGE_OK.C; no longer PRECHARGE_OK.K
- net PRECHARGE_EN: now also R1.1; no longer DIS_PRE_CHARGE_LV.6
- net PRECHARGE_OK: now also R2.1
- net V+: now also U$22.3
- net V-: now also D2.C, D3.C; no longer HVIB_HV.10, HVIB_HV.4, HVIB_HV.5, HVIB_HV.9
Routing:
- net HV-_DRY_AUX: track 94.6 -> 155.3 mm
- net V-: track 169.4 -> 124.6 mm
- net AMS_OK: track 53.7 -> 28.7 mm
- net N$42: track 0.00 -> 21.7 mm
- net HV-_ORED: track 0.00 -> 19.0 mm
- net V+: track 340.9 -> 356.5 mm
- net AMS_OK_GND: track 0.00 -> 11.2 mm
- net N$25: track 0.00 -> 10.0 mm
- net TSAL_RED_GND: track 159.6 -> 149.6 mm
- net TSAL_GRN_GND: track 164.0 -> 154.0 mm
- net ACC_LGHT: track 168.3 -> 158.3 mm
- net +12V_SAFE: track 211.0 -> 217.0 mm, vias 0 -> 1
- net N$41: track 0.00 -> 5.89 mm
- net N$27: track 0.00 -> 5.50 mm
- net PRECHARGE_OK: track 123.7 -> 129.2 mm
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- added copper zone on layer 1, net HV-_ORED
- added copper zone on layer 1, net N$44
Other:
- board text added: "EN"
- board text added: "OK"
- board text added: "PRE"

Commit message: g
Parts:
- +12V_SAFE1: device ACC-MB-R0:CHIP-LED0805 -> ACC-MB-R0:LED5MM
- moved +12V_SAFE1 0.50 mm to (175.5, 137.0), turned to 0 degrees
Connections:
- net HV-_ORED: now also +12V_SAFE1.K; no longer +12V_SAFE1.C
Routing:
- net N$41: track 5.89 -> 5.39 mm
Changed lines of the file:
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@@
 <attribute name="VALUE" x="171.325" y="129.325" size="1.27" layer="27"/>
 </element>
-<element name="+12V_SAFE1" library="ACC-MB-R0" library_urn="urn:adsk.eagle:library:13208985" package="CHIP-LED0805" package3d_urn="urn:adsk.eagle:package:15818/2" value="" x="175.5" y="137.5" smashed="yes" rot="R270">
-<attribute name="NAME" x="174.23" y="138.77" size="1.27" layer="25"/>
-<attribute name="VALUE" x="174.23" y="134.96" size="1.27" layer="27"/>
+<element name="+12V_SAFE1" library="ACC-MB-R0" library_urn="urn:adsk.eagle:library:13208985" package="LED5MM" package3d_urn="urn:adsk.eagle:package:15799/2" value="" x="175.5" y="137" smashed="yes">
+<attribute name="NAME" x="174.23" y="135.73" size="1.27" layer="25" rot="R90"/>
+<attribute name="VALUE" x="178.04" y="135.73" size="1.27" layer="27" rot="R90"/>
 </element>
 </elements>
@@
 <contactref element="INPUT_FUSE3" pad="P$2"/>
 <contactref element="U$22" pad="1"/>
-<contactref element="+12V_SAFE1" pad="C"/>
-<wire x1="176.55" y1="137.5" x2="179.5759" y2="137.5" width="1.27" layer="1"/>
+<contactref element="+12V_SAFE1" pad="K"/>
+<wire x1="176.77" y1="137" x2="179.5759" y2="137.5" width="1.27" layer="1"/>
 <wire x1="179.5759" y1="137.5" x2="179.7959" y2="137.28" width="1.27" layer="1"/>
 <wire x1="179.7959" y1="137.28" x2="176.7059" y2="140.37" width="1.27" layer="1"/>
@@
 <contactref element="R7" pad="1"/>
 <contactref element="+12V_SAFE1" pad="A"/>
-<wire x1="174.45" y1="137.5" x2="172.3" y2="135.35" width="1.27" layer="1"/>
+<wire x1="174.23" y1="137" x2="172.3" y2="135.35" width="1.27" layer="1"/>
 <wire x1="172.3" y1="135.35" x2="172.3" y2="132.5" width="1.27" layer="1"/>
 </signal>

Commit message: update
Changed lines of the file:
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@@
 <text x="107" y="9.5" size="1.778" layer="25">EN</text>
 <text x="106.5" y="3" size="1.778" layer="25">OK</text>
+<wire x1="32.5" y1="0" x2="32.5" y2="116" width="4" layer="25"/>
+<wire x1="32.5" y1="116" x2="201" y2="116" width="4" layer="25"/>
+<wire x1="201" y1="116" x2="201" y2="0.5" width="4" layer="25"/>
+<wire x1="201" y1="0.5" x2="202" y2="-0.5" width="4" layer="25"/>
+<wire x1="32.5" y1="0" x2="32.5" y2="116" width="4" layer="26"/>
+<wire x1="32.5" y1="116" x2="202" y2="116" width="4" layer="26"/>
+<wire x1="202" y1="116" x2="202" y2="0" width="4" layer="26"/>
 </plain>
 <attributes>
