File: ACC-MB/Rev3/AIRDCL/AIRDCL.brd (EAGLE design)
At the start: 172 x 64 mm, 18 parts, among them X13 5566-4

Commit message: d
Parts:
- added R4, R5: (no value), ACC-MB-R0:TO-247-2V
- moved R2 1.00 mm to (144.0, 43.0)
- moved R3 1.00 mm to (109.0, 43.0)
Connections:
- removed net N$8: R2.2, R3.1
- new net N$4: R2.2, R3.1, R4.2, R5.1
- net HV+_DRY: now also R4.1
- net N$21: now also R5.2
Routing:
- net N$8: track 37.0 -> 0.00 mm
- net N$4: track 0.00 -> 35.0 mm
- net +12V_SAFE: track 107.4 -> 139.2 mm
- net HV+_DRY: track 43.5 -> 49.2 mm
- net N$21: track 30.6 -> 29.6 mm
- added copper zone on layer 16, net HV+_DRY
- added copper zone on layer 1, net HV-_DRY
- added copper zone on layer 16, net N$21
- added copper zone on layer 16, net N$4
Other:
- outline, holes or cut-outs redrawn
- board text added: "+12V_SAFE"
- board text added: "HIGH VOLTAGE"
- board text added: "HV+ HV-AUX HV-"
- board text added: "LOW VOLTAGE"
- board text added: "REV3, BUILD1"
- board text added: "WESTERN FORMULA RACING"

Commit message: stuff
Parts:
- AIR+EN, PRECHAGE: device ACC-MB-R0:LED3MM -> ACC-MB-R0:CHIPLED_0805
- moved AIR+EN 3.64 mm to (26.5, 61.0), turned to 270 degrees
- moved LEDR3 1.80 mm to (20.5, 58.0), turned to 90 degrees
- moved LED_R4 1.12 mm to (27.5, 58.0), turned to 90 degrees
- moved PRECHAGE 1.12 mm to (21.5, 61.0), turned to 90 degrees
Connections:
- net N$2: now also PRECHAGE.C; no longer PRECHAGE.K
- net N$5: now also AIR+EN.C; no longer AIR+EN.K
Routing:
- net +12V_SAFE: track 139.2 -> 135.6 mm
- net N$2: track 3.62 -> 2.07 mm
- net N$5: track 3.32 -> 2.07 mm
Other:
- outline, holes or cut-outs redrawn
- board text added: "A1"
- board text added: "A2"
- board text added: "AIR Negative and Discharge Board Discharge R = 2x 2200 Ohm"
- board text added: "GND"
- board text added: "HV+_DRY"
- board text added: "HV-_DRY"
- board text added: "HV-_DRY_AUX"
- board text added: "NC"
- board text removed: "HV+ HV-AUX HV-"

Commit message: update
Changed lines of the file:
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@@
 <layer number="42" name="bRestrict" color="1" fill="10" visible="yes" active="yes"/>
 <layer number="43" name="vRestrict" color="2" fill="10" visible="yes" active="yes"/>
-<layer number="44" name="Drills" color="7" fill="1" visible="no" active="yes"/>
-<layer number="45" name="Holes" color="7" fill="1" visible="no" active="yes"/>
-<layer number="46" name="Milling" color="3" fill="1" visible="no" active="yes"/>
-<layer number="47" name="Measures" color="7" fill="1" visible="no" active="yes"/>
+<layer number="44" name="Drills" color="7" fill="1" visible="yes" active="yes"/>
+<layer number="45" name="Holes" color="7" fill="1" visible="yes" active="yes"/>
+<layer number="46" name="Milling" color="3" fill="1" visible="yes" active="yes"/>
+<layer number="47" name="Measures" color="7" fill="1" visible="yes" active="yes"/>
 <layer number="48" name="Document" color="7" fill="1" visible="yes" active="yes"/>
 <layer number="49" name="Reference" color="7" fill="1" visible="yes" active="yes"/>
@@
 <wire x1="82.5" y1="62" x2="93" y2="62" width="0" layer="20"/>
 <wire x1="93" y1="62" x2="95" y2="64" width="0" layer="20" curve="90"/>
-<wire x1="72" y1="68" x2="72" y2="55" width="4" layer="21"/>
-<wire x1="72" y1="55" x2="93" y2="34" width="4" layer="21"/>
-<wire x1="93" y1="34" x2="93" y2="-3" width="4" layer="21"/>
 <text x="144" y="40.5" size="1.778" layer="26" rot="MR0">AIR Negative and Discharge Board
 Discharge R = 2x 2200 Ohm</text>
+<wire x1="93" y1="1" x2="93" y2="34" width="4" layer="25"/>
+<wire x1="93" y1="34" x2="76" y2="51" width="4" layer="25"/>
+<wire x1="76" y1="51" x2="76" y2="63.5" width="4" layer="25"/>
+<wire x1="76" y1="63.5" x2="76" y2="51" width="4" layer="26"/>
+<wire x1="76" y1="51" x2="93" y2="34" width="4" layer="26"/>
+<wire x1="93" y1="34" x2="93" y2="1" width="4" layer="26"/>
 </plain>
 <attributes>
@@
 <vertex x="63.5" y="67"/>
 </polygon>
+<wire x1="57.814" y1="13.09" x2="85.58" y2="14.69" width="0" layer="19" extent="1-1"/>
+<wire x1="27.5" y1="57.05" x2="57.814" y2="13.09" width="0" layer="19" extent="1-1"/>
+<wire x1="20.5" y1="57.05" x2="27.5" y2="57.05" width="0" layer="19" extent="1-1"/>
+<wire x1="6.25" y1="42.5" x2="20.5" y2="57.05" width="0" layer="19" extent="1-1"/>
+<wire x1="2.6" y1="18.29" x2="6.25" y2="42.5" width="0" layer="19" extent="1-1"/>
+<wire x1="2.6" y1="12.79" x2="2.6" y2="18.29" width="0" layer="19" extent="1-1"/>
 </signal>
 <signal name="N$5">
