File: ACC-MB/Rev3/AIRDCR/AIRDCR.brd (EAGLE design)
At the start: 172 x 64 mm, 18 parts, among them X13 5566-4

Commit message: d
Parts:
- added R4, R5: (no value), ACC-MB-R0:TO-247-2V
- moved R2 6.50 mm to (55.5, 42.5)
- moved R3 6.50 mm to (32.5, 42.5)
- turned U$8 to 270 degrees
- turned U$9 to 90 degrees
Connections:
- removed net N$8: R2.2, R3.1
- new net N$4: R2.2, R3.1, R4.2, R5.1
- net HV+_WET: now also R4.1
- net N$21: now also R5.2
Routing:
- net N$8: track 36.0 -> 0.00 mm
- net N$4: track 0.00 -> 23.0 mm
- net N$21: track 50.4 -> 40.1 mm
- net HV+_WET: track 29.6 -> 36.1 mm
- net HV+_DRY: track 145.7 -> 140.0 mm
- added copper zone on layer 1, net HV+_DRY
- added copper zone on layer 16, net HV+_WET
- added copper zone on layer 16, net N$21
- added copper zone on layer 16, net N$4
Other:
- outline, holes or cut-outs redrawn
- board text added: "HIGH VOLTAGE"
- board text added: "HV+"
- board text added: "HV+_DRY"
- board text added: "HV+_WET"
- board text added: "LOW VOLTAGE"
- board text added: "REV3, BUILD1"
- board text added: "WESTERN FORMULA RACING"

Commit message: stuff
Parts:
- AIR+EN, PRECHAGE: device ACC-MB-R0:LED3MM -> ACC-MB-R0:CHIPLED_0805
- moved LED_R3 59.0 mm to (163.5, 60.5)
- moved PRECHAGE 58.8 mm to (168.0, 60.5), turned to 90 degrees
- moved X13 1.00 mm to (79.0, 48.0)
- moved AIR+EN 0.71 mm to (138.0, 62.0), turned to 270 degrees
- moved LED_R4 0.71 mm to (143.0, 62.0)
Connections:
- net N$2: now also PRECHAGE.C; no longer PRECHAGE.K
- net N$5: now also AIR+EN.C; no longer AIR+EN.K
Routing:
- net PRECHARGE: track 99.6 -> 147.9 mm
- net COIL_X1: track 82.5 -> 92.9 mm
- net N$5: track 6.56 -> 3.00 mm
- net HV+_DRY: track 140.0 -> 139.0 mm
Other:
- outline, holes or cut-outs redrawn
- board text added: "AIR Positive and Precharge Board Precharge R = 2x 620 Ohm"
- board text added: "NC"

Commit message: g
Parts:
- moved AIR+EN 1.12 mm to (137.0, 61.5)
- moved LED_R4 1.12 mm to (142.0, 61.5)
Routing:
- net COIL_X1: track 92.9 -> 84.4 mm, vias 0 -> 1
Changed lines of the file:
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@@
 <setting verticaltext="up"/>
 </settings>
-<grid distance="0.5" unitdist="mm" unit="mm" style="dots" multiple="1" display="yes" altdistance="0.5" altunitdist="mm" altunit="mm"/>
+<grid distance="0.125" unitdist="mm" unit="mm" style="dots" multiple="1" display="yes" altdistance="0.5" altunitdist="mm" altunit="mm"/>
 <layers>
 <layer number="1" name="Top" color="4" fill="1" visible="yes" active="yes"/>
@@
 <attribute name="VALUE" x="68.19" y="47.985" size="1.27" layer="27"/>
 </element>
-<element name="AIR+EN" library="ACC-MB-R0" library_urn="urn:adsk.eagle:library:13208985" package="CHIPLED_0805" package3d_urn="urn:adsk.eagle:package:15821/2" value="" x="138" y="62" smashed="yes" rot="R270">
-<attribute name="NAME" x="137.905" y="59.381" size="1.27" layer="25" ratio="10"/>
-<attribute name="VALUE" x="136.349" y="60.095" size="1.27" layer="27" ratio="10" rot="R270"/>
-</element>
-<element name="LED_R4" library="ACC-MB-R0" library_urn="urn:adsk.eagle:library:13208985" package="R0805" package3d_urn="urn:adsk.eagle:package:13209583/1" value="" x="143" y="62" smashed="yes" rot="R180">
-<attribute name="SPICEPREFIX" value="R" x="143" y="62" size="1.778" layer="27" rot="R180" display="off"/>
-<attribute name="VALUE" x="143.635" y="64.54" size="1.27" layer="27" rot="R180"/>
+<element name="AIR+EN" library="ACC-MB-R0" library_urn="urn:adsk.eagle:library:13208985" package="CHIPLED_0805" package3d_urn="urn:adsk.eagle:package:15821/2" value="" x="137" y="61.5" smashed="yes" rot="R270">
+<attribute name="NAME" x="136.905" y="58.881" size="1.27" layer="25" ratio="10"/>
+<attribute name="VALUE" x="135.349" y="59.595" size="1.27" layer="27" ratio="10" rot="R270"/>
+</element>
+<element name="LED_R4" library="ACC-MB-R0" library_urn="urn:adsk.eagle:library:13208985" package="R0805" package3d_urn="urn:adsk.eagle:package:13209583/1" value="" x="142" y="61.5" smashed="yes" rot="R180">
+<attribute name="SPICEPREFIX" value="R" x="142" y="61.5" size="1.778" layer="27" rot="R180" display="off"/>
+<attribute name="VALUE" x="142.635" y="64.04" size="1.27" layer="27" rot="R180"/>
 </element>
 <element name="U$4" library="ACC-MB-R0" library_urn="urn:adsk.eagle:library:13208985" package="G81C335" package3d_urn="urn:adsk.eagle:package:14396596/2" value="G81C335" x="27" y="3.5" smashed="yes" rot="MR180"/>
@@
 <contactref element="AIR+EN" pad="A"/>
 <contactref element="U$3" pad="2"/>
-<wire x1="162.97" y1="18.48" x2="162.97" y2="25.15" width="1" layer="16"/>
-<wire x1="145.09" y1="52.91" x2="124.314" y2="52.91" width="1.27" layer="16"/>
+<wire x1="163.095" y1="14.895" x2="163.095" y2="25.025" width="1.27" layer="16"/>
+<wire x1="145.09" y1="52.91" x2="134" y2="52.91" width="1.27" layer="16"/>
+<wire x1="134" y1="52.91" x2="124.314" y2="52.91" width="1.27" layer="16"/>
 <wire x1="124.314" y1="52.91" x2="122.314" y2="51.29" width="1.27" layer="16"/>
 <wire x1="149.15" y1="48.85" x2="149.15" y2="36" width="1.27" layer="16"/>
@@
 <wire x1="154.15" y1="30.47" x2="157.62" y2="27" width="1.27" layer="16"/>
 <wire x1="157.62" y1="27" x2="161.12" y2="27" width="1.27" layer="16"/>
-<wire x1="161.12" y1="27" x2="162.97" y2="25.15" width="1.27" layer="16"/>
-<wire x1="165.2" y1="12.79" x2="162.97" y2="15.02" width="1.016" layer="16"/>
-<wire x1="162.97" y1="15.02" x2="162.97" y2="18.48" width="1.016" layer="16"/>
-<wire x1="136.95" y1="62" x2="133.024" y2="62" width="0.2" layer="1"/>
-<wire x1="133.024" y1="62" x2="122.314" y2="51.29" width="0.2" layer="1"/>
+<wire x1="161.12" y1="27" x2="163.095" y2="25.025" width="1.27" layer="16"/>
+<wire x1="165.2" y1="12.79" x2="163.095" y2="14.895" width="1.27" layer="16"/>
+<wire x1="135.95" y1="61.5" x2="134" y2="61.5" width="0.2" layer="1"/>
+<via x="134" y="61.5" extent="1-16" drill="0.35"/>
+<wire x1="134" y1="61.5" x2="134" y2="52.91" width="0.2" layer="16"/>
 </signal>
 <signal name="N$3">
@@
 <contactref element="U$3" pad="5"/>
 <contactref element="U$1" pad="X2"/>
-<wire x1="143.95" y1="62" x2="114.186" y2="51.29" width="0" layer="19" extent="1-1"/>
 </signal>
 <signal name="N$5">
 <contactref element="LED_R4" pad="2"/>
 <contactref element="AIR+EN" pad="C"/>
-<wire x1="139.05" y1="62" x2="142.05" y2="62" width="0.2" layer="1"/>
+<wire x1="138.05" y1="61.5" x2="141.05" y2="61.5" width="0.2" layer="1"/>
 </signal>
 <signal name="HV+_DRY" class="2">
@@
 <wire x1="154.5" y1="2" x2="161.5" y2="9" width="1.016" layer="16"/>
 <wire x1="161.5" y1="9" x2="168" y2="9" width="1.016" layer="16"/>
-<wire x1="169.27" y1="55.27" x2="169.25" y2="55.25" width="0.2" layer="1"/>
-<wire x1="169.25" y1="55.25" x2="163.5" y2="49.5" width="0.2" layer="1"/>
+<wire x1="169.27" y1="55.27" x2="163.5" y2="49.5" width="0.2" layer="1"/>
 <wire x1="163.5" y1="49.5" x2="163.5" y2="27" width="0.2" layer="1"/>
 <wire x1="163.5" y1="27" x2="167.5" y2="23" width="0.2" layer="1"/>
 <wire x1="167.5" y1="23" x2="167.5" y2="14.69" width="0.2" layer="1"/>
 <wire x1="167.5" y1="14.69" x2="169.4" y2="12.79" width="0.2" layer="1"/>
-<wire x1="169.25" y1="55.25" x2="169.25" y2="60.3" width="0.2" layer="1"/>
+<wire x1="169.27" y1="55.27" x2="169.25" y2="55.29" width="0.2" layer="1"/>
+<wire x1="169.25" y1="60.3" x2="169.25" y2="55.29" width="0.2" layer="1"/>
 <wire x1="169.25" y1="60.3" x2="169.05" y2="60.5" width="0.2" layer="1"/>
 </signal>

Commit message: update
Changed lines of the file:
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@@
 Precharge R = 2x 620 Ohm
 </text>
-<wire x1="73" y1="-1" x2="73" y2="21" width="4" layer="112"/>
-<wire x1="73" y1="21" x2="88" y2="21" width="4" layer="112"/>
-<wire x1="88" y1="21" x2="88" y2="51" width="4" layer="112"/>
-<wire x1="88" y1="51" x2="103" y2="51" width="4" layer="112"/>
-<wire x1="103" y1="51" x2="103" y2="66" width="4" layer="112"/>
+<wire x1="73.125" y1="0.375" x2="73.125" y2="19.875" width="4" layer="25"/>
+<wire x1="73.125" y1="19.875" x2="88.5" y2="35.25" width="4" layer="25"/>
+<wire x1="88.5" y1="35.25" x2="88.5" y2="49.625" width="4" layer="25"/>
+<wire x1="88.5" y1="49.625" x2="102.75" y2="63.875" width="4" layer="25"/>
+<wire x1="102.75" y1="63.875" x2="88.5" y2="49.625" width="4" layer="26"/>
+<wire x1="88.5" y1="49.625" x2="88.5" y2="35.25" width="4" layer="26"/>
+<wire x1="88.5" y1="35.25" x2="73.125" y2="19.875" width="4" layer="26"/>
+<wire x1="73.125" y1="19.875" x2="73.125" y2="0.375" width="4" layer="26"/>
 </plain>
 <attributes>
@@
 <contactref element="U$3" pad="5"/>
 <contactref element="U$1" pad="X2"/>
+<wire x1="158.25" y1="43" x2="162.55" y2="60.5" width="0" layer="19" extent="1-1"/>
+<wire x1="142.95" y1="61.5" x2="162.55" y2="60.5" width="0" layer="19" extent="1-1"/>
+<wire x1="152.6" y1="18.29" x2="158.25" y2="43" width="0" layer="19" extent="1-1"/>
+<wire x1="152.6" y1="12.79" x2="152.6" y2="18.29" width="0" layer="19" extent="1-1"/>
+<wire x1="114.186" y1="51.29" x2="142.95" y2="61.5" width="0" layer="19" extent="1-1"/>
+<wire x1="85.42" y1="7.31" x2="114.186" y2="51.29" width="0" layer="19" extent="1-1"/>
 </signal>
 <signal name="N$5">
