File: ACC-MB/Rev3/AIRDCR/AIRDCR.sch (EAGLE design)
At the start: 18 parts, among them X13 5566-4

Commit message: d
Parts:
- added R4, R5: (no value), ACC-MB-R0:RMG100-V
Connections:
- removed net N$8: R2.2, R3.1
- new net N$4: R2.2, R3.1, R4.2, R5.1
- net HV+_WET: now also R4.1
- net N$21: now also R5.2
Changed lines of the file:
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@@
 </class>
 <class number="2" name="HV" width="1.27" drill="0">
-<clearance class="0" value="1.5"/>
-<clearance class="1" value="1.5"/>
-<clearance class="2" value="1.5"/>
+<clearance class="0" value="1.8"/>
+<clearance class="1" value="1.8"/>
+<clearance class="2" value="1.8"/>
 </class>
 </classes>
@@
 <part name="U$8" library="ACC-MB-R0" library_urn="urn:adsk.eagle:library:13208985" deviceset="RA-T2X-25E" device="" package3d_urn="urn:adsk.eagle:package:15294014/2"/>
 <part name="U$9" library="ACC-MB-R0" library_urn="urn:adsk.eagle:library:13208985" deviceset="RA-T2X-25E" device="" package3d_urn="urn:adsk.eagle:package:15294014/2"/>
+<part name="R4" library="ACC-MB-R0" library_urn="urn:adsk.eagle:library:13208985" deviceset="RMG100" device="-V" package3d_urn="urn:adsk.eagle:package:13209920/2"/>
+<part name="R5" library="ACC-MB-R0" library_urn="urn:adsk.eagle:library:13208985" deviceset="RMG100" device="-V" package3d_urn="urn:adsk.eagle:package:13209920/2"/>
 </parts>
 <sheets>
@@
 <instance part="U$8" gate="G$1" x="236.22" y="177.8" smashed="yes"/>
 <instance part="U$9" gate="G$1" x="254" y="177.8" smashed="yes"/>
+<instance part="R4" gate="G$1" x="246.38" y="170.18" smashed="yes">
+<attribute name="NAME" x="242.57" y="171.5516" size="1.778" layer="95"/>
+<attribute name="VALUE" x="242.57" y="167.259" size="1.778" layer="96"/>
+</instance>
+<instance part="R5" gate="G$1" x="259.08" y="170.18" smashed="yes">
+<attribute name="NAME" x="255.27" y="171.5516" size="1.778" layer="95"/>
+<attribute name="VALUE" x="255.27" y="167.259" size="1.778" layer="96"/>
+</instance>
 </instances>
 <busses>
@@
 <net name="N$21" class="2">
 <segment>
-<wire x1="273.05" y1="172.72" x2="264.16" y2="172.72" width="0.1524" layer="91"/>
+<wire x1="273.05" y1="172.72" x2="266.7" y2="172.72" width="0.1524" layer="91"/>
 <pinref part="U$4" gate="G$1" pin="COM"/>
+<wire x1="266.7" y1="172.72" x2="264.16" y2="172.72" width="0.1524" layer="91"/>
 <wire x1="264.16" y1="172.72" x2="262.89" y2="172.72" width="0.1524" layer="91"/>
 <wire x1="273.05" y1="172.72" x2="274.32" y2="172.72" width="0.1524" layer="91"/>
@@
 <pinref part="R3" gate="G$1" pin="2"/>
 <junction x="264.16" y="172.72"/>
+<pinref part="R5" gate="G$1" pin="2"/>
+<wire x1="264.16" y1="170.18" x2="266.7" y2="170.18" width="0.1524" layer="91"/>
+<wire x1="266.7" y1="170.18" x2="266.7" y2="172.72" width="0.1524" layer="91"/>
+<junction x="266.7" y="172.72"/>
 </segment>
 </net>
@@
 </segment>
 </net>
-<net name="N$8" class="2">
-<segment>
-<wire x1="251.46" y1="172.72" x2="254" y2="172.72" width="0.1524" layer="91"/>
-<pinref part="R2" gate="G$1" pin="2"/>
-<pinref part="R3" gate="G$1" pin="1"/>
-</segment>
-</net>
 <net name="HV+_WET" class="2">
 <segment>
@@
 <wire x1="228.6" y1="172.72" x2="231.14" y2="172.72" width="0.1524" layer="91"/>
 <pinref part="X13" gate="-4" pin="S"/>
-<wire x1="231.14" y1="172.72" x2="241.3" y2="172.72" width="0.1524" layer="91"/>
+<wire x1="231.14" y1="172.72" x2="238.76" y2="172.72" width="0.1524" layer="91"/>
+<wire x1="238.76" y1="172.72" x2="241.3" y2="172.72" width="0.1524" layer="91"/>
 <wire x1="228.6" y1="175.26" x2="231.14" y2="175.26" width="0.1524" layer="91"/>
 <wire x1="231.14" y1="175.26" x2="231.14" y2="172.72" width="0.1524" layer="91"/>
@@
 <label x="231.14" y="172.72" size="1.778" layer="95"/>
 <pinref part="R2" gate="G$1" pin="1"/>
-</segment>
-</net>
+<pinref part="R4" gate="G$1" pin="1"/>
+<wire x1="241.3" y1="170.18" x2="238.76" y2="170.18" width="0.1524" layer="91"/>
+<wire x1="238.76" y1="170.18" x2="238.76" y2="172.72" width="0.1524" layer="91"/>
+<junction x="238.76" y="172.72"/>
+</segment>
+</net>
+<net name="N$4" class="0">
+<segment>
+<pinref part="R4" gate="G$1" pin="2"/>
+<pinref part="R5" gate="G$1" pin="1"/>
+<wire x1="251.46" y1="170.18" x2="254" y2="170.18" width="0.1524" layer="91"/>
+<wire x1="251.46" y1="172.72" x2="254" y2="172.72" width="0.1524" layer="91"/>
+<pinref part="R2" gate="G$1" pin="2"/>
+<pinref part="R3" gate="G$1" pin="1"/>
+<wire x1="251.46" y1="170.18" x2="251.46" y2="172.72" width="0.1524" layer="91"/>
+<junction x="251.46" y="170.18"/>
+<junction x="251.46" y="172.72"/>
+</segment>
+</net>

Commit message: stuff
Parts:
- AIR+EN, PRECHAGE: device ACC-MB-R0:LED3MM -> ACC-MB-R0:LEDCHIPLED_0805
Changed lines of the file:
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@@
 <part name="GND1" library="Main" library_urn="urn:adsk.eagle:library:14107900" deviceset="GND" device=""/>
 <part name="X13" library="ACC-MB-R0" library_urn="urn:adsk.eagle:library:13208985" deviceset="5566-4" device="" package3d_urn="urn:adsk.eagle:package:14396878/3"/>
-<part name="AIR+EN" library="ACC-MB-R0" library_urn="urn:adsk.eagle:library:13208985" deviceset="LED" device="3MM" package3d_urn="urn:adsk.eagle:package:15797/1"/>
+<part name="AIR+EN" library="ACC-MB-R0" library_urn="urn:adsk.eagle:library:13208985" deviceset="LED" device="CHIPLED_0805" package3d_urn="urn:adsk.eagle:package:15821/2"/>
 <part name="LED_R4" library="ACC-MB-R0" library_urn="urn:adsk.eagle:library:13208985" deviceset="R-US_" device="R0805" package3d_urn="urn:adsk.eagle:package:13209583/1"/>
 <part name="GND3" library="ACC-MB-R0" library_urn="urn:adsk.eagle:library:13208985" deviceset="GND" device=""/>
 <part name="GND5" library="ACC-MB-R0" library_urn="urn:adsk.eagle:library:13208985" deviceset="GND" device=""/>
 <part name="U$4" library="ACC-MB-R0" library_urn="urn:adsk.eagle:library:13208985" deviceset="G81C335" device="" package3d_urn="urn:adsk.eagle:package:14396596/2"/>
-<part name="PRECHAGE" library="ACC-MB-R0" library_urn="urn:adsk.eagle:library:13208985" deviceset="LED" device="3MM" package3d_urn="urn:adsk.eagle:package:15797/1"/>
+<part name="PRECHAGE" library="ACC-MB-R0" library_urn="urn:adsk.eagle:library:13208985" deviceset="LED" device="CHIPLED_0805" package3d_urn="urn:adsk.eagle:package:15821/2"/>
 <part name="LED_R3" library="ACC-MB-R0" library_urn="urn:adsk.eagle:library:13208985" deviceset="R-US_" device="R0805" package3d_urn="urn:adsk.eagle:package:13209583/1"/>
 <part name="GND6" library="ACC-MB-R0" library_urn="urn:adsk.eagle:library:13208985" deviceset="GND" device=""/>
