File: ACC-MB/Rev3/DCDCDC-r2/DCDCDC-R2.brd (EAGLE design)
At the start: 172 x 64 mm, 38 parts, among them P1330-102H 39uH

Commit message: d
Parts:
- added R10, R27, R7, R9: CRM2512-JW-102ELF, ACC-MB-R0:R2512
- moved CFILTER_1 1.00 mm to (29.5, 29.5)
- moved U$8 1.00 mm to (61.0, 33.0)
- moved CFILTER_2 0.75 mm to (18.5, 29.5)
Connections:
- new net N$12: R27.2, R7.1
- new net N$13: R7.2, R9.1
- new net N$14: R10.1, R9.2
- net V+: now also R10.2
- net V-: now also R27.1
Routing:
- net V-: track 60.1 -> 81.7 mm
- net N$13: track 0.00 -> 12.0 mm
- net V+: track 24.0 -> 30.2 mm
- net N$14: track 0.00 -> 3.40 mm
- net N$12: track 0.00 -> 3.40 mm
- net N$7: track 25.4 -> 27.0 mm
Other:
- outline, holes or cut-outs redrawn
- board text added: "+VOUT GND"
- board text added: "DC/DC CONVERTER 600W 400V TO 13.8V"
- board text added: "DCDC OUTPUT"
- board text added: "HIGH VOLTAGE"
- board text added: "HV+ HV-"
- board text added: "HV- HV+"
- board text added: "LOW VOLTAGE"
- board text added: "OUTPUT ENABLED"
- board text added: "REV3, BUILD1"
- board text added: "VICOR FAULT"
- board text added: "WESTERN FORMULA RACING"

Commit message: stuff
Parts:
- added LED4: (no value), ACC-MB-R0:CHIPLED_0805
- added R11: (no value), ACC-MB-R0:R0805
- LED1, LED2, LED3: device ACC-MB-R0:LED3MM -> ACC-MB-R0:CHIPLED_0805
Connections:
- new net N$11: LED4.C, R11.2
- net N$5: now also LED1.C; no longer LED1.K
- net N$6: now also LED2.C; no longer LED2.K
- net N$7: now also LED4.A
- net N$9: now also LED3.C; no longer LED3.K
- net V-: now also R11.1
Routing:
- net N$7: track 27.0 -> 35.8 mm
- net N$6: track 2.63 -> 8.34 mm, vias 0 -> 1
- net N$9: track 2.13 -> 5.18 mm, vias 0 -> 1
- net N$11: track 0.00 -> 3.00 mm
- net N$5: track 2.87 -> 4.58 mm, vias 0 -> 1
- net N$10: track 98.8 -> 99.1 mm, vias 0 -> 1
Other:
- board text added: "+12V"
- board text added: "EN"
- board text added: "FAN"
- board text added: "GND"
- board text removed: "+VOUT GND"
Changed lines of the file:
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@@
 </text>
 <text x="62" y="2" size="3.81" layer="21">WESTERN   FORMULA   RACING</text>
-<text x="150" y="33" size="1.778" layer="21">+VOUT
-GND</text>
 <text x="3" y="22" size="2.54" layer="21">HV+   HV-</text>
 <wire x1="52" y1="15" x2="52" y2="23" width="4" layer="21"/>
@@
 <wire x1="3" y1="0" x2="0" y2="3" width="0" layer="20" curve="-90"/>
 <text x="16" y="6" size="1.778" layer="26" rot="MR0">HV-  HV+</text>
+<text x="141" y="17" size="1.778" layer="25">+12V</text>
+<text x="141" y="12" size="1.778" layer="25">GND</text>
+<text x="168" y="23" size="1.778" layer="25">EN</text>
+<text x="143" y="39" size="1.778" layer="25">GND</text>
+<text x="148" y="43" size="1.778" layer="25" rot="R90">+12V</text>
+<text x="126" y="10" size="1.778" layer="25">FAN</text>
 </plain>
 <attributes>
@@
 <attribute name="NAME" x="121.75" y="40" size="1.27" layer="21" rot="R270"/>
 </element>
-<element name="LED1" library="ACC-MB-R0" library_urn="urn:adsk.eagle:library:13208985" package="LED3MM" package3d_urn="urn:adsk.eagle:package:15797/1" value="" x="122" y="50.5" smashed="yes">
+<element name="LED1" library="ACC-MB-R0" library_urn="urn:adsk.eagle:library:13208985" package="CHIPLED_0805" package3d_urn="urn:adsk.eagle:package:15821/2" value="" x="122" y="50.5" smashed="yes">
 <attribute name="VALUE" x="123.905" y="48.849" size="1.27" layer="27" ratio="10"/>
 </element>
@@
 <attribute name="VALUE" x="47.03" y="19.03" size="1.27" layer="21"/>
 </element>
-<element name="LED2" library="ACC-MB-R0" library_urn="urn:adsk.eagle:library:13208985" package="LED3MM" package3d_urn="urn:adsk.eagle:package:15797/1" value="" x="111" y="58" smashed="yes" rot="R270">
+<element name="LED2" library="ACC-MB-R0" library_urn="urn:adsk.eagle:library:13208985" package="CHIPLED_0805" package3d_urn="urn:adsk.eagle:package:15821/2" value="" x="111" y="58" smashed="yes" rot="R270">
 <attribute name="VALUE" x="109.349" y="56.095" size="1.27" layer="27" ratio="10" rot="R270"/>
 </element>
@@
 <attribute name="VALUE" x="45.925" y="9.925" size="1.27" layer="27" rot="R180"/>
 </element>
-<element name="LED3" library="ACC-MB-R0" library_urn="urn:adsk.eagle:library:13208985" package="LED3MM" package3d_urn="urn:adsk.eagle:package:15797/1" value="" x="106" y="58" smashed="yes" rot="R270">
+<element name="LED3" library="ACC-MB-R0" library_urn="urn:adsk.eagle:library:13208985" package="CHIPLED_0805" package3d_urn="urn:adsk.eagle:package:15821/2" value="" x="106" y="58" smashed="yes" rot="R270">
 <attribute name="VALUE" x="104.349" y="56.095" size="1.27" layer="27" ratio="10" rot="R270"/>
 </element>
@@
 </element>
 <element name="U$13" library="ACC-MB-R0" library_urn="urn:adsk.eagle:library:13208985" package="39-28-1103" package3d_urn="urn:adsk.eagle:package:14745616/3" value="39-28-1103" x="161" y="43" smashed="yes" rot="R180">
-<attribute name="NAME" x="155.285" y="49.985" size="1.27" layer="25" rot="R180"/>
-<attribute name="VALUE" x="171.16" y="49.985" size="1.27" layer="27" rot="R180"/>
+<attribute name="NAME" x="155.285" y="43.985" size="1.27" layer="25" rot="R180"/>
+<attribute name="VALUE" x="171.16" y="43.985" size="1.27" layer="27" rot="R180"/>
 </element>
 <element name="U$9" library="ACC-MB-R0" library_urn="urn:adsk.eagle:library:13208985" package="15-24-6100" package3d_urn="urn:adsk.eagle:package:14396594/3" value="15-24-6100" x="11" y="15.54" smashed="yes">
@@
 <attribute name="NAME" x="5.095" y="29.54" size="1.27" layer="26" rot="MR270"/>
 <attribute name="SPICEPREFIX" value="R" x="7" y="27" size="1.778" layer="28" rot="MR270" display="off"/>
+</element>
+<element name="LED4" library="ACC-MB-R0" library_urn="urn:adsk.eagle:library:13208985" package="CHIPLED_0805" package3d_urn="urn:adsk.eagle:package:15821/2" value="" x="30" y="10" smashed="yes" rot="R90">
+<attribute name="NAME" x="29.619" y="11.905" size="1.27" layer="25" ratio="10" rot="R90"/>
+<attribute name="VALUE" x="31.651" y="11.905" size="1.27" layer="27" ratio="10" rot="R90"/>
+</element>
+<element name="R11" library="ACC-MB-R0" library_urn="urn:adsk.eagle:library:13208985" package="R0805" package3d_urn="urn:adsk.eagle:package:13209583/1" value="" x="25" y="10" smashed="yes">
+<attribute name="NAME" x="24.365" y="11.27" size="1.27" layer="25"/>
+<attribute name="SPICEPREFIX" value="R" x="25" y="10" size="1.778" layer="27" display="off"/>
+<attribute name="VALUE" x="24.365" y="7.46" size="1.27" layer="27"/>
 </element>
 </elements>
@@
 <wire x1="18.25" y1="24" x2="18.5" y2="25.575" width="3" layer="1"/>
 <wire x1="31.5" y1="21.5" x2="29" y2="24" width="3" layer="1"/>
+<contactref element="R11" pad="1"/>
+<wire x1="19.4" y1="12.79" x2="24.05" y2="10" width="0" layer="19" extent="1-1"/>
 </signal>
 <signal name="+12V">
@@
 <signal name="N$5">
 <contactref element="R4" pad="2"/>
-<contactref element="LED1" pad="K"/>
-<wire x1="123.27" y1="50.5" x2="124.22" y2="49.55" width="0.2" layer="16"/>
-<wire x1="124.22" y1="49.55" x2="125.75" y2="49.55" width="0.2" layer="16"/>
+<contactref element="LED1" pad="C"/>
+<wire x1="125.75" y1="49.55" x2="124.45" y2="49.55" width="0.2" layer="16"/>
+<wire x1="124.45" y1="49.55" x2="124" y2="50" width="0.2" layer="16"/>
+<via x="124" y="50" extent="1-16" drill="0.35"/>
+<wire x1="124" y1="50" x2="123.55" y2="50" width="0.2" layer="1"/>
+<wire x1="123.55" y1="50" x2="122" y2="51.55" width="0.2" layer="1"/>
 </signal>
 <signal name="N$6">
 <contactref element="R5" pad="2"/>
-<contactref element="LED2" pad="K"/>
-<wire x1="111.25" y1="54.2" x2="111.25" y2="56.48" width="0.2" layer="16"/>
-<wire x1="111.25" y1="56.48" x2="111" y2="56.73" width="0.2" layer="16"/>
+<contactref element="LED2" pad="C"/>
+<wire x1="112.05" y1="58" x2="111" y2="59.05" width="0.2" layer="1"/>
+<wire x1="111" y1="59.05" x2="111" y2="60" width="0.2" layer="1"/>
+<via x="111" y="60" extent="1-16" drill="0.35"/>
+<wire x1="111" y1="60" x2="111.25" y2="59.75" width="0.2" layer="16"/>
+<wire x1="111.25" y1="59.75" x2="111.25" y2="54.2" width="0.2" layer="16"/>
 </signal>
 <signal name="+12V_FUSED1">
@@
 <contactref element="U$8" pad="FT"/>
 <contactref element="R16" pad="2"/>
-<wire x1="39.8" y1="21.8" x2="39.8" y2="7.5" width="0.3048" layer="1"/>
+<wire x1="39.8" y1="21.8" x2="39.8" y2="10" width="0.3048" layer="1"/>
+<wire x1="39.8" y1="10" x2="39.8" y2="7.5" width="0.3048" layer="1"/>
 <wire x1="40.55" y1="6.75" x2="39.8" y2="7.5" width="0.3048" layer="1"/>
 <wire x1="39.8" y1="21.8" x2="42" y2="24" width="0.3048" layer="1"/>
@@
 <wire x1="42" y1="28" x2="41.13" y2="28.87" width="0.3048" layer="1"/>
 <wire x1="41.13" y1="28.87" x2="37.81" y2="28.87" width="0.3048" layer="1"/>
+<contactref element="LED4" pad="A"/>
+<wire x1="31.05" y1="10" x2="39.8" y2="10" width="0.2" layer="1"/>
 </signal>
 <signal name="N$9">
 <contactref element="R6" pad="2"/>
-<contactref element="LED3" pad="K"/>
-<wire x1="105.75" y1="54.7" x2="105.75" y2="56.48" width="0.2" layer="16"/>
-<wire x1="105.75" y1="56.48" x2="106" y2="56.73" width="0.2" layer="16"/>
+<contactref element="LED3" pad="C"/>
+<wire x1="107.05" y1="58" x2="107.05" y2="56.95" width="0.2" layer="1"/>
+<wire x1="107.05" y1="56.95" x2="108" y2="56" width="0.2" layer="1"/>
+<via x="108" y="56" extent="1-16" drill="0.35"/>
+<wire x1="108" y1="56" x2="107.05" y2="56" width="0.2" layer="16"/>
+<wire x1="107.05" y1="56" x2="105.75" y2="54.7" width="0.2" layer="16"/>
 </signal>
 <signal name="N$10">
 <contactref element="OK3" pad="3"/>
 <contactref element="LED3" pad="A"/>
-<wire x1="106" y1="59.27" x2="105" y2="60.27" width="0.2" layer="16"/>
-<wire x1="105" y1="60.27" x2="75" y2="60.27" width="0.2" layer="16"/>
+<wire x1="75" y1="60.27" x2="105" y2="60.27" width="0.2" layer="16"/>
 <wire x1="75" y1="60.27" x2="70" y2="55.27" width="0.2" layer="16"/>
 <wire x1="70" y1="55.27" x2="59" y2="44.27" width="0.3048" layer="16"/>
-<wire x1="59" y1="3" x2="56.58" y2="3" width="0.3048" layer="16"/>
-<wire x1="56.58" y1="3" x2="55.81" y2="2.23" width="0.3048" layer="16"/>
-<wire x1="59" y1="44.27" x2="59" y2="3" width="0.3048" layer="16"/>
+<wire x1="59" y1="4" x2="57.23" y2="2.23" width="0.3048" layer="16"/>
+<wire x1="57.23" y1="2.23" x2="55.81" y2="2.23" width="0.3048" layer="16"/>
+<wire x1="59" y1="44.27" x2="59" y2="4" width="0.3048" layer="16"/>
+<via x="105" y="60.27" extent="1-16" drill="0.35"/>
+<wire x1="105" y1="60.27" x2="105" y2="58.05" width="0.2" layer="1"/>
+<wire x1="105" y1="58.05" x2="104.95" y2="58" width="0.2" layer="1"/>
 </signal>
 <signal name="+12V_FUSED">
@@
 <wire x1="7" y1="33.2" x2="7" y2="29.8" width="2.54" layer="16"/>
 </signal>
+<signal name="N$11">
+<contactref element="R11" pad="2"/>
+<contactref element="LED4" pad="C"/>
+<wire x1="25.95" y1="10" x2="28.95" y2="10" width="0.2" layer="1"/>
+</signal>
 </signals>

Commit message: g
Parts:
- moved LED4 0.75 mm to (30.0, 9.25)
- moved R11 0.75 mm to (25.0, 9.25)
- moved U$5 0.12 mm to (123.3, 58.3)
Routing:
- net V-: track 81.7 -> 147.6 mm
- net V+_FUSED: track 25.7 -> 72.1 mm
- net N$3: track 28.2 -> 64.5 mm
- net V+: track 30.2 -> 44.1 mm
- net GND: track 11.8 -> 17.2 mm
- net DCDC_OUT: track 0.00 -> 4.70 mm

Commit message: update
Changed lines of the file:
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@@
 <layer number="44" name="Drills" color="7" fill="1" visible="no" active="yes"/>
 <layer number="45" name="Holes" color="7" fill="1" visible="no" active="yes"/>
-<layer number="46" name="Milling" color="3" fill="1" visible="no" active="yes"/>
+<layer number="46" name="Milling" color="3" fill="1" visible="yes" active="yes"/>
 <layer number="47" name="Measures" color="7" fill="1" visible="no" active="yes"/>
 <layer number="48" name="Document" color="7" fill="1" visible="yes" active="yes"/>
@@
 <wire x1="3" y1="0" x2="169" y2="0" width="0" layer="20"/>
 <wire x1="172" y1="3" x2="172" y2="61" width="0" layer="20"/>
-<wire x1="52" y1="-2" x2="52" y2="15" width="4" layer="21"/>
 <dimension x1="50" y1="56" x2="54" y2="56" x3="52" y3="59" textsize="3.81" layer="21"/>
 <text x="23.25" y="60.5" size="2.54" layer="21">HIGH VOLTAGE</text>
@@
 <text x="62" y="2" size="3.81" layer="21">WESTERN   FORMULA   RACING</text>
 <text x="3" y="22" size="2.54" layer="21">HV+   HV-</text>
-<wire x1="52" y1="15" x2="52" y2="23" width="4" layer="21"/>
-<wire x1="52" y1="23" x2="52" y2="43" width="4" layer="21"/>
-<wire x1="52" y1="43" x2="52" y2="66" width="4" layer="21"/>
-<wire x1="52" y1="23" x2="44" y2="23" width="4" layer="21"/>
-<wire x1="44" y1="23" x2="42" y2="21" width="4" layer="21"/>
-<wire x1="42" y1="21" x2="42" y2="17" width="4" layer="21"/>
-<wire x1="42" y1="17" x2="44" y2="15" width="4" layer="21"/>
-<wire x1="44" y1="15" x2="52" y2="15" width="4" layer="21"/>
-<wire x1="51" y1="51" x2="44" y2="51" width="4" layer="21"/>
-<wire x1="44" y1="51" x2="42" y2="49" width="4" layer="21"/>
-<wire x1="42" y1="48" x2="42" y2="45" width="4" layer="21"/>
-<wire x1="42" y1="45" x2="44" y2="43" width="4" layer="21"/>
-<wire x1="44" y1="43" x2="52" y2="43" width="4" layer="21"/>
 <text x="98" y="7.25" size="1.778" layer="25">REV3, BUILD1</text>
 <text x="108" y="47.75" size="1.778" layer="25" rot="R90">VICOR
@@
 <text x="148" y="43" size="1.778" layer="25" rot="R90">+12V</text>
 <text x="126" y="10" size="1.778" layer="25">FAN</text>
+<wire x1="52" y1="63.625" x2="52" y2="0.75" width="4" layer="25"/>
+<wire x1="52.125" y1="0.875" x2="52.125" y2="63.75" width="4" layer="26"/>
 </plain>
 <attributes>
@@
 <element name="U$8" library="ACC-MB-R0" library_urn="urn:adsk.eagle:library:13208985" package="VICOR_CHIP_HEATSINK" package3d_urn="urn:adsk.eagle:package:13209498/4" value="VICOR_DCM_CHIP" x="61" y="33" smashed="yes">
 <attribute name="NAME" x="47.03" y="45.7" size="1.27" layer="21"/>
-<attribute name="VALUE" x="47.03" y="19.03" size="1.27" layer="21"/>
+<attribute name="VALUE" x="73.72" y="26.28" size="1.27" layer="21" rot="R90"/>
 </element>
 <element name="LED2" library="ACC-MB-R0" library_urn="urn:adsk.eagle:library:13208985" package="CHIPLED_0805" package3d_urn="urn:adsk.eagle:package:15821/2" value="" x="111" y="58" smashed="yes" rot="R270">
