File: PDM-GLV/PDM.brd (EAGLE design)
At the start: 82.5 x 101.6 mm, 10 parts

Commit message: g
Routing:
- net CH11: track 0.00 -> 21.1 mm
- net CH10: track 0.00 -> 21.1 mm
- net CH8: track 13.3 -> 31.6 mm
Other:
- board text removed: "Expansion Relays"
Changed lines of the file:
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@@
 <vertex x="42.275" y="88.6"/>
 </polygon>
-<wire x1="23.4" y1="14.1" x2="50.1" y2="-12.2" width="0.1524" layer="47"/>
-<wire x1="50.1" y1="-12.2" x2="55.1" y2="14" width="0.1524" layer="47"/>
-<wire x1="50.1" y1="-12.2" x2="71.6" y2="-12.2" width="0.1524" layer="47"/>
-<text x="50.9" y="-12" size="1.778" layer="47">Expansion Relays</text>
 </plain>
 <attributes>
@@
 <contactref element="CH7" pad="L1"/>
 <contactref element="CH7" pad="L2"/>
-<wire x1="79.245" y1="2.45" x2="79.245" y2="8.755" width="3" layer="16"/>
-<wire x1="79.245" y1="8.755" x2="79" y2="9" width="3" layer="16"/>
-<wire x1="79" y1="9" x2="79.045" y2="9" width="3" layer="16"/>
-<wire x1="79.045" y1="9" x2="79.245" y2="8.8" width="3" layer="16"/>
 <polygon width="1.5" layer="1" rank="4">
 <vertex x="46" y="62"/>
@@
 <vertex x="86" y="-3"/>
 </polygon>
+<wire x1="79.245" y1="2.45" x2="75.176" y2="2.45" width="2.54" layer="1"/>
+<wire x1="75.176" y1="2.45" x2="75.055" y2="2.571" width="2.54" layer="1"/>
+<wire x1="75.055" y1="8.8" x2="79.245" y2="8.8" width="2.54" layer="16"/>
+<wire x1="79.245" y1="8.8" x2="79.245" y2="2.45" width="2.54" layer="16"/>
+<wire x1="79.245" y1="2.45" x2="75.055" y2="2.45" width="2.54" layer="16"/>
+<wire x1="75.055" y1="2.45" x2="75.055" y2="8.8" width="2.54" layer="16"/>
 </signal>
 <signal name="CH10">
@@
 <vertex x="45" y="-2"/>
 </polygon>
+<wire x1="66.675" y1="8.8" x2="70.865" y2="8.8" width="2.54" layer="16"/>
+<wire x1="70.865" y1="8.8" x2="70.865" y2="2.45" width="2.54" layer="16"/>
+<wire x1="70.865" y1="2.45" x2="66.675" y2="2.45" width="2.54" layer="16"/>
+<wire x1="66.675" y1="2.45" x2="66.675" y2="8.8" width="2.54" layer="16"/>
 </signal>
 <signal name="CH11">
@@
 <vertex x="64" y="-2"/>
 </polygon>
+<wire x1="58.295" y1="8.8" x2="58.295" y2="2.45" width="2.54" layer="16"/>
+<wire x1="58.295" y1="2.45" x2="62.485" y2="2.45" width="2.54" layer="16"/>
+<wire x1="62.485" y1="2.45" x2="62.485" y2="8.8" width="2.54" layer="16"/>
+<wire x1="62.485" y1="8.8" x2="58.295" y2="8.8" width="2.54" layer="16"/>
 </signal>
 <signal name="COMMON">

Commit message: update
Other:
- board text added: "1 2 3"
- board text added: "A B C D E F"
Changed lines of the file:
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@@
 <vertex x="42.275" y="88.6"/>
 </polygon>
+<text x="38" y="47" size="3.81" layer="25">A
+B
+C
+D
+E
+F</text>
+<text x="70" y="31" size="3.81" layer="25">1
+2
+3</text>
 </plain>
 <attributes>
@@
 </drawing>
 <compatibility>
+<note version="6.3" minversion="6.2.2" severity="warning">
+Since Version 6.2.2 text objects can contain more than one line,
+which will not be processed correctly with this version.
+</note>
 <note version="8.2" severity="warning">
 Since Version 8.2, EAGLE supports online libraries. The ids
